File: kicad/qPCR-kicad/module/photoarray/qPCR-photoarray.kicad_pcb (KiCad board)
At the start: 2 copper layers, 34 parts, among them U1 TF31-18S-0.5SH(800), U2 TF31-18S-0.5SH(800)

Commit message: add slide0
Parts:
- moved D1 0.75 mm to (117.0, 63.0)
- moved D10 0.75 mm to (155.0, 63.0)
- moved D11 0.75 mm to (162.0, 63.0)
- moved D12 0.75 mm to (164.0, 63.0)
- moved D13 0.75 mm to (171.0, 63.0)
- moved D14 0.75 mm to (173.0, 63.0)
- moved D15 0.75 mm to (180.0, 63.0)
- moved D16 0.75 mm to (182.0, 63.0)
- moved D17 0.75 mm to (117.2, 85.0)
- moved D18 0.75 mm to (118.8, 85.0)
- moved D19 0.75 mm to (126.2, 85.0)
- moved D2 0.75 mm to (119.0, 63.0)
- moved D20 0.75 mm to (127.8, 85.0)
- moved D21 0.75 mm to (135.2, 85.0)
- moved D22 0.75 mm to (136.8, 85.0)
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Routing:
- net GND: track 136.5 -> 8.12 mm, vias 6 -> 0
- net OUT16: track 76.2 -> 0.00 mm
- net OUT32: track 75.8 -> 0.00 mm
- net OUT31: track 72.6 -> 0.00 mm
- net OUT15: track 72.5 -> 0.00 mm
- net OUT14: track 66.8 -> 0.00 mm
- net OUT30: track 66.4 -> 0.00 mm
- net OUT29: track 63.2 -> 0.00 mm
- net OUT13: track 63.2 -> 0.00 mm
- net OUT12: track 57.5 -> 0.00 mm
- net OUT28: track 57.0 -> 0.00 mm
- net OUT11: track 53.9 -> 0.00 mm
- net OUT27: track 53.8 -> 0.00 mm
- net OUT10: track 51.7 -> 0.00 mm
- net OUT9: track 48.0 -> 0.00 mm
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Other:
- board outline added: 2.1 x 2.1 mm
