File: kicad/Ninja-qPCR/batch2/photo_mux/photo_mux_ADG706BRUZ-ND/qPCR-photo_mux_ADG706BRUZ-ND.sch (KiCad schematic (older format))
At the start: 23 parts

Commit message: sync
Parts:
- removed U?: Conn_02x05, symbol Ninja-qPCR:Conn_02x05
- added J? (x2): Conn_01x05_Male, symbol Connector:Conn_01x05_Male
- C1, C2, C3, C4: renamed from C?; footprint (none) -> Capacitors_SMD:C_0603_HandSoldering
- JP1, JP2, JP3: renamed from JP?; footprint (none) -> Jumper:SolderJumper-3_P2.0mm_Open_TrianglePad1.0x1.5mm
- N_PD1, N_PD2, S_PD1, S_PD2: footprint (none) -> Ninja-qPCR:Con_2x05
- U1: renamed from U?; footprint RU_28_ADI -> (none)
- gave numbers to parts that had none: 8
Connections:
- net +10V: now also J?.2 (Pin_2)
- net -10V: now also J?.3 (Pin_3)
- net ADDRESSA0: now also U1.17 (A0), J?.4 (Pin_4); no longer U4.17 (A0)
- net ADDRESSA1: now also U1.16 (A1), J?.3 (Pin_3); no longer U4.16 (A1)
- net ADDRESSA2: now also U1.15 (A2), J?.2 (Pin_2); no longer U4.15 (A2)
- net ADDRESSA3: now also U1.14 (A3), J?.1 (Pin_1); no longer U4.14 (A3)
- net GND: now also U4.12 (GND), J?.1 (Pin_1); no longer U1.12 (GND)
- net MUX_SELECT: now also J?.5 (Pin_5)
- net MUX_SELECT_INV: now also U1.18 (EN); no longer U4.18 (EN)
- net PD_MUX_OUT: now also J?.5 (Pin_5)
- net PD_MUX_OUT2: now also U1.28 (D); no longer U4.28 (D)
- net S_PD1_OUT1: now also U1.19 (S1); no longer U4.19 (S1)
- net S_PD1_OUT10: now also U1.10 (S10); no longer U4.10 (S10)
- net S_PD1_OUT11: now also U1.9 (S11); no longer U4.9 (S11)
- net S_PD1_OUT12: now also U1.8 (S12); no longer U4.8 (S12)
- net S_PD1_OUT13: now also U1.7 (S13); no longer U4.7 (S13)
- net S_PD1_OUT14: now also U1.6 (S14); no longer U4.6 (S14)
- net S_PD1_OUT15: now also U1.5 (S15); no longer U4.5 (S15)
- net S_PD1_OUT16: now also U1.4 (S16); no longer U4.4 (S16)
- net S_PD1_OUT2: now also U1.20 (S2); no longer U4.20 (S2)
- net S_PD1_OUT3: now also U1.21 (S3); no longer U4.21 (S3)
- net S_PD1_OUT4: now also U1.22 (S4); no longer U4.22 (S4)
- net S_PD1_OUT5: now also U1.23 (S5); no longer U4.23 (S5)
- net S_PD1_OUT6: now also U1.24 (S6); no longer U4.24 (S6)
- net S_PD1_OUT7: now also U1.25 (S7); no longer U4.25 (S7)
- net S_PD1_OUT8: now also U1.26 (S8); no longer U4.26 (S8)
- net S_PD1_OUT9: now also U1.11 (S9); no longer U4.11 (S9)
- net VCC_LOGIC: now also J?.4 (Pin_4)
- net VDD: now also U4.1 (VDD); no longer U1.1 (VDD)
- net VSS: now also U4.27 (VSS); no longer U1.27 (VSS)

Commit message: sync
Parts:
- removed C3, C4: C, Capacitors_SMD:C_0603_HandSoldering, symbol Device:C
- J1, J2: renamed from J?; footprint (none) -> Pin_Headers:Pin_Header_Straight_1x05_Pitch2.54mm
- R1, R2, R3, R4, R5, R6: footprint (none) -> Resistors_SMD:R_0603_HandSoldering
- U1: footprint (none) -> Ninja-qPCR:ADG706BRUZ
- U3: footprint SOT95P280X145-5N -> Ninja-qPCR:SN74LVC1G04DBVR
- U4: footprint RU_28_ADI -> Ninja-qPCR:ADG706BRUZ
Changed lines of the file:
@@
 F 0 "U3" H 3200 4617 50  0000 C CNN
 F 1 "SN74LVC1G04DBVR" H 3200 4526 50  0000 C CNN
-F 2 "SOT95P280X145-5N" H 3200 4150 50  0001 L BNN
+F 2 "Ninja-qPCR:SN74LVC1G04DBVR" H 3200 4150 50  0001 L BNN
 F 3 "IPC-7351B" H 3200 4150 50  0001 L BNN
 F 4 "1.45mm" H 3200 4150 50  0001 L BNN "Field4"
@@
 F 0 "U4" H 9350 1887 60  0000 C CNN
 F 1 "ADG706BRUZ" H 9350 1781 60  0000 C CNN
-F 2 "RU_28_ADI" H 9350 1740 60  0001 C CNN
+F 2 "Ninja-qPCR:ADG706BRUZ" H 9350 1740 60  0001 C CNN
 F 3 "" H 8550 1400 60  0000 C CNN
 	1    8550 1400
@@
 F 0 "U1" H 9350 4487 60  0000 C CNN
 F 1 "ADG706BRUZ" H 9350 4381 60  0000 C CNN
-F 2 "" H 9350 4340 60  0001 C CNN
+F 2 "Ninja-qPCR:ADG706BRUZ" H 9350 4340 60  0001 C CNN
 F 3 "" H 8550 4000 60  0000 C CNN
 	1    8550 4000
@@
 F 0 "U1" H 4950 7287 60  0000 C CNN
 F 1 "ADG706BRUZ" H 4950 7181 60  0000 C CNN
-F 2 "" H 4950 7140 60  0001 C CNN
+F 2 "Ninja-qPCR:ADG706BRUZ" H 4950 7140 60  0001 C CNN
 F 3 "" H 4150 6800 60  0000 C CNN
 	2    4150 6800
@@
 Wire Wire Line
 	4150 5950 4150 5800
-Text GLabel 4700 5350 0    50   Input ~ 0
-+10V
-Text GLabel 4700 5950 0    50   Input ~ 0
-GND
-$Comp
-L Device:C C3
-U 1 1 5F5A298B
-P 4850 5650
-F 0 "C3" H 4965 5696 50  0000 L CNN
-F 1 "C" H 4965 5605 50  0000 L CNN
-F 2 "Capacitors_SMD:C_0603_HandSoldering" H 4888 5500 50  0001 C CNN
-F 3 "~" H 4850 5650 50  0001 C CNN
-	1    4850 5650
-	1    0    0    -1
-$EndComp
-Wire Wire Line
-	4700 5350 4850 5350
-Wire Wire Line
-	4850 5350 4850 5500
-Wire Wire Line
-	4700 5950 4850 5950
-Wire Wire Line
-	4850 5950 4850 5800
-Text GLabel 5350 5350 0    50   Input ~ 0
--10V
-Text GLabel 5350 5950 0    50   Input ~ 0
-GND
-$Comp
-L Device:C C4
-U 1 1 5F5A2997
-P 5500 5650
-F 0 "C4" H 5615 5696 50  0000 L CNN
-F 1 "C" H 5615 5605 50  0000 L CNN
-F 2 "Capacitors_SMD:C_0603_HandSoldering" H 5538 5500 50  0001 C CNN
-F 3 "~" H 5500 5650 50  0001 C CNN
-	1    5500 5650
-	1    0    0    -1
-$EndComp
-Wire Wire Line
-	5500 5500 5500 5350
-Wire Wire Line
-	5500 5350 5350 5350
-Wire Wire Line
-	5350 5950 5500 5950
-Wire Wire Line
-	5500 5950 5500 5800
 Text GLabel 3900 1700 0    50   Input ~ 0
 +10V
@@
 F 0 "U4" H 2550 7287 60  0000 C CNN
 F 1 "ADG706BRUZ" H 2550 7181 60  0000 C CNN
-F 2 "RU_28_ADI" H 2550 7140 60  0001 C CNN
+F 2 "Ninja-qPCR:ADG706BRUZ" H 2550 7140 60  0001 C CNN
 F 3 "" H 1750 6800 60  0000 C CNN
 	2    1750 6800
@@
 F 0 "R3" H 4120 2846 50  0000 L CNN
 F 1 "R" H 4120 2755 50  0000 L CNN
-F 2 "" V 3980 2800 50  0001 C CNN
+F 2 "Resistors_SMD:R_0603_HandSoldering" V 3980 2800 50  0001 C CNN
 F 3 "~" H 4050 2800 50  0001 C CNN
 	1    4050 2800
@@
 F 0 "R2" H 4120 2446 50  0000 L CNN
 F 1 "R" H 4120 2355 50  0000 L CNN
-F 2 "" V 3980 2400 50  0001 C CNN
+F 2 "Resistors_SMD:R_0603_HandSoldering" V 3980 2400 50  0001 C CNN
 F 3 "~" H 4050 2400 50  0001 C CNN
 	1    4050 2400
@@
 F 0 "R1" H 4120 2046 50  0000 L CNN
 F 1 "R" H 4120 1955 50  0000 L CNN
-F 2 "" V 3980 2000 50  0001 C CNN
+F 2 "Resistors_SMD:R_0603_HandSoldering" V 3980 2000 50  0001 C CNN
 F 3 "~" H 4050 2000 50  0001 C CNN
 	1    4050 2000
@@
 F 0 "R6" H 4770 2846 50  0000 L CNN
 F 1 "R" H 4770 2755 50  0000 L CNN
-F 2 "" V 4630 2800 50  0001 C CNN
+F 2 "Resistors_SMD:R_0603_HandSoldering" V 4630 2800 50  0001 C CNN
 F 3 "~" H 4700 2800 50  0001 C CNN
 	1    4700 2800
@@
 F 0 "R5" H 4770 2446 50  0000 L CNN
 F 1 "R" H 4770 2355 50  0000 L CNN
-F 2 "" V 4630 2400 50  0001 C CNN
+F 2 "Resistors_SMD:R_0603_HandSoldering" V 4630 2400 50  0001 C CNN
 F 3 "~" H 4700 2400 50  0001 C CNN
 	1    4700 2400
@@
 F 0 "R4" H 4770 2046 50  0000 L CNN
 F 1 "R" H 4770 1955 50  0000 L CNN
-F 2 "" V 4630 2000 50  0001 C CNN
+F 2 "Resistors_SMD:R_0603_HandSoldering" V 4630 2000 50  0001 C CNN
 F 3 "~" H 4700 2000 50  0001 C CNN
 	1    4700 2000
@@
 	6950 4300 6800 4300
 $Comp
-L Connector:Conn_01x05_Male J?
+L Connector:Conn_01x05_Male J1
 U 1 1 5F5A772F
 P 950 2250
-F 0 "J?" H 1058 2631 50  0000 C CNN
+F 0 "J1" H 1058 2631 50  0000 C CNN
 F 1 "Conn_01x05_Male" H 1058 2540 50  0000 C CNN
-F 2 "" H 950 2250 50  0001 C CNN
+F 2 "Pin_Headers:Pin_Header_Straight_1x05_Pitch2.54mm" H 950 2250 50  0001 C CNN
 F 3 "~" H 950 2250 50  0001 C CNN
 	1    950  2250
@@
 $EndComp
 $Comp
-L Connector:Conn_01x05_Male J?
+L Connector:Conn_01x05_Male J2
 U 1 1 5F5A8B7D
 P 950 3050
-F 0 "J?" H 1058 3431 50  0000 C CNN
+F 0 "J2" H 1058 3431 50  0000 C CNN
 F 1 "Conn_01x05_Male" H 1058 3340 50  0000 C CNN
-F 2 "" H 950 3050 50  0001 C CNN
+F 2 "Pin_Headers:Pin_Header_Straight_1x05_Pitch2.54mm" H 950 3050 50  0001 C CNN
 F 3 "~" H 950 3050 50  0001 C CNN
 	1    950  3050

Commit message: sync
Parts:
- C1, C2: value C -> 0.1uF
Changed lines of the file:
@@
 P 3500 5650
 F 0 "C1" H 3615 5696 50  0000 L CNN
-F 1 "C" H 3615 5605 50  0000 L CNN
+F 1 "0.1uF" H 3615 5605 50  0000 L CNN
 F 2 "Capacitors_SMD:C_0603_HandSoldering" H 3538 5500 50  0001 C CNN
 F 3 "~" H 3500 5650 50  0001 C CNN
@@
 P 4150 5650
 F 0 "C2" H 4265 5696 50  0000 L CNN
-F 1 "C" H 4265 5605 50  0000 L CNN
+F 1 "0.1uF" H 4265 5605 50  0000 L CNN
 F 2 "Capacitors_SMD:C_0603_HandSoldering" H 4188 5500 50  0001 C CNN
 F 3 "~" H 4150 5650 50  0001 C CNN
