File: kicad/Ninja-qPCR/batch2/photo_mux/photo_mux_ADG731BSUZ/qPCR-photo_mux_ADG731BSUZ.sch (KiCad schematic (older format))
At the start: 17 parts

Commit message: sync
Parts:
- removed U?: Conn_02x05, symbol Ninja-qPCR:Conn_02x05
- added J? (x2): Conn_01x05_Male, symbol Connector:Conn_01x05_Male
Connections:
- net +10V: now also J?.2 (Pin_2)
- net -10V: now also J?.3 (Pin_3)
- net GND: now also J?.1 (Pin_1)
- net PD_MUX_OUT: now also J?.5 (Pin_5)
- net PD_MUX_SPI_MOSI: now also J?.4 (Pin_4)
- net PD_MUX_SPL_SCLK: now also J?.3 (Pin_3)
- net PD_MUX_SYNC: now also J?.5 (Pin_5)
- net VCC_LOGIC: now also J?.4 (Pin_4)
Changed lines of the file:
@@
 	1    0    0    -1
 $EndComp
-Text GLabel 1900 2050 0    50   Input ~ 0
-GND
-Text GLabel 1900 2150 0    50   Input ~ 0
+Text GLabel 1250 1200 2    50   Input ~ 0
+GND
+Text GLabel 1250 1300 2    50   Input ~ 0
 +10V
-Text GLabel 1900 2250 0    50   Input ~ 0
+Text GLabel 1250 1400 2    50   Input ~ 0
 -10V
-Text GLabel 1900 2350 0    50   Input ~ 0
+Text GLabel 1250 1500 2    50   Input ~ 0
 VCC_LOGIC
-Text GLabel 1900 2450 0    50   Input ~ 0
+Text GLabel 1250 1600 2    50   Input ~ 0
 PD_MUX_OUT
 Wire Wire Line
-	2100 2050 1900 2050
-Wire Wire Line
-	1900 2150 2100 2150
-Wire Wire Line
-	2100 2250 1900 2250
-Wire Wire Line
-	1900 2350 2100 2350
-Wire Wire Line
-	2100 2450 1900 2450
-Wire Wire Line
-	1900 2550 2100 2550
-Wire Wire Line
-	2100 2650 1900 2650
-Wire Wire Line
-	1900 2750 2100 2750
-Wire Wire Line
-	2100 2850 1900 2850
-$Comp
-L Ninja-qPCR:Conn_02x05 U?
-U 1 1 5F51FB4B
-P 2300 2050
-F 0 "U?" H 2619 1661 50  0000 L CNN
-F 1 "Conn_02x05" H 2619 1570 50  0000 L CNN
-F 2 "" H 2100 2150 50  0001 C CNN
-F 3 "" H 2100 2150 50  0001 C CNN
-	1    2300 2050
-	1    0    0    -1
-$EndComp
-Wire Wire Line
-	1900 2950 2100 2950
+	1050 1200 1250 1200
+Wire Wire Line
+	1250 1300 1050 1300
+Wire Wire Line
+	1050 1400 1250 1400
+Wire Wire Line
+	1250 1500 1050 1500
+Wire Wire Line
+	1050 1600 1250 1600
+Wire Wire Line
+	1250 1950 1050 1950
+Wire Wire Line
+	1050 2050 1250 2050
+Wire Wire Line
+	1250 2150 1050 2150
+Wire Wire Line
+	1050 2250 1250 2250
+Wire Wire Line
+	1250 2350 1050 2350
 $Comp
 L Ninja-qPCR:ADG731BSUZ U?
@@
 Wire Wire Line
 	6950 1050 6800 1050
-Text GLabel 1900 2750 0    50   Input ~ 0
+Text GLabel 1250 2150 2    50   Input ~ 0
 PD_MUX_SPL_SCLK
-Text GLabel 1900 2850 0    50   Input ~ 0
+Text GLabel 1250 2250 2    50   Input ~ 0
 PD_MUX_SPI_MOSI
-Text GLabel 1900 2950 0    50   Input ~ 0
+Text GLabel 1250 2350 2    50   Input ~ 0
 PD_MUX_SYNC
-NoConn ~ 1900 2550
+NoConn ~ 1250 1950
 Text GLabel 6800 1150 0    50   Input ~ 0
 PD_MUX_SPI_MOSI
@@
 Wire Wire Line
 	8550 4350 8700 4350
-NoConn ~ 1900 2650
+NoConn ~ 1250 2050
 Text GLabel 1750 4600 0    50   Input ~ 0
 +10V
@@
 Wire Wire Line
 	6950 5100 6750 5100
+$Comp
+L Connector:Conn_01x05_Male J?
+U 1 1 5F5948A2
+P 850 1400
+F 0 "J?" H 958 1781 50  0000 C CNN
+F 1 "Conn_01x05_Male" H 958 1690 50  0000 C CNN
+F 2 "" H 850 1400 50  0001 C CNN
+F 3 "~" H 850 1400 50  0001 C CNN
+	1    850  1400
+	1    0    0    -1
+$EndComp
+$Comp
+L Connector:Conn_01x05_Male J?
+U 1 1 5F5950CF
+P 850 2150
+F 0 "J?" H 958 2531 50  0000 C CNN
+F 1 "Conn_01x05_Male" H 958 2440 50  0000 C CNN
+F 2 "" H 850 2150 50  0001 C CNN
+F 3 "~" H 850 2150 50  0001 C CNN
+	1    850  2150
+	1    0    0    -1
+$EndComp
 $EndSCHEMATC

Commit message: sync
Parts:
- C1, C2: renamed from C?; footprint (none) -> Capacitors_SMD:C_0805_HandSoldering
- J1, J2: renamed from J?; footprint (none) -> Pin_Headers:Pin_Header_Straight_1x05_Pitch2.54mm
- JP1, JP2: renamed from JP?; footprint (none) -> Jumper:SolderJumper-3_P2.0mm_Open_TrianglePad1.0x1.5mm
- N_PD1, N_PD2, S_PD1, S_PD2: footprint (none) -> Ninja-qPCR:Con_2x05
- R1, R2, R3, R4, R5, R6: renamed from R?; footprint (none) -> Resistors_SMD:R_0603_HandSoldering
- U1: renamed from U?; footprint SU_48_ADI -> Ninja-qPCR:ADG731BSUZ
Connections:
- net +10V: no longer C1.1
- net -10V: no longer C2.1
- net VDD: now also C1.1
- net VSS: now also C2.1
Changed lines of the file:
@@
 F 0 "N_PD1" H 10650 -200 50  0000 L CNN
 F 1 "Conn_02x05" H 10650 -300 50  0000 L CNN
-F 2 "" H 10550 950 50  0001 C CNN
+F 2 "Ninja-qPCR:Con_2x05" H 10550 950 50  0001 C CNN
 F 3 "" H 10550 950 50  0001 C CNN
 	1    10750 850
@@
 F 0 "N_PD2" H 10650 1150 50  0000 L CNN
 F 1 "Conn_02x05" H 10650 1050 50  0000 L CNN
-F 2 "" H 10550 2300 50  0001 C CNN
+F 2 "Ninja-qPCR:Con_2x05" H 10550 2300 50  0001 C CNN
 F 3 "" H 10550 2300 50  0001 C CNN
 	1    10750 2200
@@
 F 0 "S_PD2" H 10650 4200 50  0000 L CNN
 F 1 "Conn_02x05" H 10650 4100 50  0000 L CNN
-F 2 "" H 10550 5350 50  0001 C CNN
+F 2 "Ninja-qPCR:Con_2x05" H 10550 5350 50  0001 C CNN
 F 3 "" H 10550 5350 50  0001 C CNN
 	1    10750 5250
@@
 F 0 "S_PD1" H 10600 2700 50  0000 L CNN
 F 1 "Conn_02x05" H 10600 2600 50  0000 L CNN
-F 2 "" H 10500 3850 50  0001 C CNN
+F 2 "Ninja-qPCR:Con_2x05" H 10500 3850 50  0001 C CNN
 F 3 "" H 10500 3850 50  0001 C CNN
 	1    10700 3750
@@
 	1250 2350 1050 2350
 $Comp
-L Ninja-qPCR:ADG731BSUZ U?
+L Ninja-qPCR:ADG731BSUZ U1
 U 1 1 5F54A8CC
 P 8550 1050
-F 0 "U?" H 9350 1537 60  0000 C CNN
+F 0 "U1" H 9350 1537 60  0000 C CNN
 F 1 "ADG731BSUZ" H 9350 1431 60  0000 C CNN
-F 2 "SU_48_ADI" H 9350 1390 60  0001 C CNN
+F 2 "Ninja-qPCR:ADG731BSUZ" H 9350 1390 60  0001 C CNN
 F 3 "" H 8550 1050 60  0000 C CNN
 	1    8550 1050
@@
 $EndComp
 $Comp
-L Ninja-qPCR:ADG731BSUZ U?
+L Ninja-qPCR:ADG731BSUZ U1
 U 2 1 5F54DA1F
 P 8550 5100
-F 0 "U?" H 9350 5587 60  0000 C CNN
+F 0 "U1" H 9350 5587 60  0000 C CNN
 F 1 "ADG731BSUZ" H 9350 5481 60  0000 C CNN
-F 2 "SU_48_ADI" H 9350 5440 60  0001 C CNN
+F 2 "Ninja-qPCR:ADG731BSUZ" H 9350 5440 60  0001 C CNN
 F 3 "" H 8550 5100 60  0000 C CNN
 	2    8550 5100
@@
 NoConn ~ 1250 2050
 Text GLabel 1750 4600 0    50   Input ~ 0
-+10V
+VDD
 Text GLabel 2600 4600 0    50   Input ~ 0
--10V
-$Comp
-L Device:C C?
+VSS
+$Comp
+L Device:C C1
 U 1 1 5F579FC2
 P 1850 4850
-F 0 "C?" H 1965 4896 50  0000 L CNN
+F 0 "C1" H 1965 4896 50  0000 L CNN
 F 1 "C" H 1965 4805 50  0000 L CNN
-F 2 "" H 1888 4700 50  0001 C CNN
+F 2 "Capacitors_SMD:C_0805_HandSoldering" H 1888 4700 50  0001 C CNN
 F 3 "~" H 1850 4850 50  0001 C CNN
 	1    1850 4850
@@
 $EndComp
 $Comp
-L Device:C C?
+L Device:C C2
 U 1 1 5F57B129
 P 2700 4850
-F 0 "C?" H 2815 4896 50  0000 L CNN
+F 0 "C2" H 2815 4896 50  0000 L CNN
 F 1 "C" H 2815 4805 50  0000 L CNN
-F 2 "" H 2738 4700 50  0001 C CNN
+F 2 "Capacitors_SMD:C_0805_HandSoldering" H 2738 4700 50  0001 C CNN
 F 3 "~" H 2700 4850 50  0001 C CNN
 	1    2700 4850
@@
 GND
 $Comp
-L Device:R R?
+L Device:R R3
 U 1 1 5F582087
 P 3450 4850
-F 0 "R?" H 3520 4896 50  0000 L CNN
+F 0 "R3" H 3520 4896 50  0000 L CNN
 F 1 "R" H 3520 4805 50  0000 L CNN
-F 2 "" V 3380 4850 50  0001 C CNN
+F 2 "Resistors_SMD:R_0603_HandSoldering" V 3380 4850 50  0001 C CNN
 F 3 "~" H 3450 4850 50  0001 C CNN
 	1    3450 4850
@@
 $EndComp
 $Comp
-L Device:R R?
+L Device:R R2
 U 1 1 5F582D94
 P 3450 4450
-F 0 "R?" H 3520 4496 50  0000 L CNN
+F 0 "R2" H 3520 4496 50  0000 L CNN
 F 1 "R" H 3520 4405 50  0000 L CNN
-F 2 "" V 3380 4450 50  0001 C CNN
+F 2 "Resistors_SMD:R_0603_HandSoldering" V 3380 4450 50  0001 C CNN
 F 3 "~" H 3450 4450 50  0001 C CNN
 	1    3450 4450
@@
 $EndComp
 $Comp
-L Device:R R?
+L Device:R R1
 U 1 1 5F583415
 P 3450 4050
-F 0 "R?" H 3520 4096 50  0000 L CNN
+F 0 "R1" H 3520 4096 50  0000 L CNN
 F 1 "R" H 3520 4005 50  0000 L CNN
-F 2 "" V 3380 4050 50  0001 C CNN
+F 2 "Resistors_SMD:R_0603_HandSoldering" V 3380 4050 50  0001 C CNN
 F 3 "~" H 3450 4050 50  0001 C CNN
 	1    3450 4050
@@
 GND
 $Comp
-L Device:R R?
+L Device:R R6
 U 1 1 5F585C52
 P 4300 4850
-F 0 "R?" H 4370 4896 50  0000 L CNN
+F 0 "R6" H 4370 4896 50  0000 L CNN
 F 1 "R" H 4370 4805 50  0000 L CNN
-F 2 "" V 4230 4850 50  0001 C CNN
+F 2 "Resistors_SMD:R_0603_HandSoldering" V 4230 4850 50  0001 C CNN
 F 3 "~" H 4300 4850 50  0001 C CNN
 	1    4300 4850
@@
 $EndComp
 $Comp
-L Device:R R?
+L Device:R R5
 U 1 1 5F585C58
 P 4300 4450
-F 0 "R?" H 4370 4496 50  0000 L CNN
+F 0 "R5" H 4370 4496 50  0000 L CNN
 F 1 "R" H 4370 4405 50  0000 L CNN
-F 2 "" V 4230 4450 50  0001 C CNN
+F 2 "Resistors_SMD:R_0603_HandSoldering" V 4230 4450 50  0001 C CNN
 F 3 "~" H 4300 4450 50  0001 C CNN
 	1    4300 4450
@@
 $EndComp
 $Comp
-L Device:R R?
+L Device:R R4
 U 1 1 5F585C5E
 P 4300 4050
-F 0 "R?" H 4370 4096 50  0000 L CNN
+F 0 "R4" H 4370 4096 50  0000 L CNN
 F 1 "R" H 4370 4005 50  0000 L CNN
-F 2 "" V 4230 4050 50  0001 C CNN
+F 2 "Resistors_SMD:R_0603_HandSoldering" V 4230 4050 50  0001 C CNN
 F 3 "~" H 4300 4050 50  0001 C CNN
 	1    4300 4050
@@
 GND
 $Comp
-L Jumper:Jumper_3_Open JP?
+L Jumper:Jumper_3_Open JP1
 U 1 1 5F5E99B2
 P 5500 2950
-F 0 "JP?" H 5500 3174 50  0000 C CNN
+F 0 "JP1" H 5500 3174 50  0000 C CNN
 F 1 "Jumper_3_Open" H 5500 3083 50  0000 C CNN
-F 2 "" H 5500 2950 50  0001 C CNN
+F 2 "Jumper:SolderJumper-3_P2.0mm_Open_TrianglePad1.0x1.5mm" H 5500 2950 50  0001 C CNN
 F 3 "~" H 5500 2950 50  0001 C CNN
 	1    5500 2950
@@
 -3.33V
 $Comp
-L Jumper:Jumper_3_Open JP?
+L Jumper:Jumper_3_Open JP2
 U 1 1 5F5EACA3
 P 5500 4100
-F 0 "JP?" H 5500 4324 50  0000 C CNN
+F 0 "JP2" H 5500 4324 50  0000 C CNN
 F 1 "Jumper_3_Open" H 5500 4233 50  0000 C CNN
-F 2 "" H 5500 4100 50  0001 C CNN
+F 2 "Jumper:SolderJumper-3_P2.0mm_Open_TrianglePad1.0x1.5mm" H 5500 4100 50  0001 C CNN
 F 3 "~" H 5500 4100 50  0001 C CNN
 	1    5500 4100
@@
 	6950 5100 6750 5100
 $Comp
-L Connector:Conn_01x05_Male J?
+L Connector:Conn_01x05_Male J1
 U 1 1 5F5948A2
 P 850 1400
-F 0 "J?" H 958 1781 50  0000 C CNN
+F 0 "J1" H 958 1781 50  0000 C CNN
 F 1 "Conn_01x05_Male" H 958 1690 50  0000 C CNN
-F 2 "" H 850 1400 50  0001 C CNN
+F 2 "Pin_Headers:Pin_Header_Straight_1x05_Pitch2.54mm" H 850 1400 50  0001 C CNN
 F 3 "~" H 850 1400 50  0001 C CNN
 	1    850  1400
@@
 $EndComp
 $Comp
-L Connector:Conn_01x05_Male J?
+L Connector:Conn_01x05_Male J2
 U 1 1 5F5950CF
 P 850 2150
-F 0 "J?" H 958 2531 50  0000 C CNN
+F 0 "J2" H 958 2531 50  0000 C CNN
 F 1 "Conn_01x05_Male" H 958 2440 50  0000 C CNN
-F 2 "" H 850 2150 50  0001 C CNN
+F 2 "Pin_Headers:Pin_Header_Straight_1x05_Pitch2.54mm" H 850 2150 50  0001 C CNN
 F 3 "~" H 850 2150 50  0001 C CNN
 	1    850  2150

Commit message: sync
Parts:
- C1, C2: value C -> 0.1uF?
Changed lines of the file:
@@
 P 1850 4850
 F 0 "C1" H 1965 4896 50  0000 L CNN
-F 1 "C" H 1965 4805 50  0000 L CNN
+F 1 "0.1uF?" H 1965 4805 50  0000 L CNN
 F 2 "Capacitors_SMD:C_0805_HandSoldering" H 1888 4700 50  0001 C CNN
 F 3 "~" H 1850 4850 50  0001 C CNN
@@
 P 2700 4850
 F 0 "C2" H 2815 4896 50  0000 L CNN
-F 1 "C" H 2815 4805 50  0000 L CNN
+F 1 "0.1uF?" H 2815 4805 50  0000 L CNN
 F 2 "Capacitors_SMD:C_0805_HandSoldering" H 2738 4700 50  0001 C CNN
 F 3 "~" H 2700 4850 50  0001 C CNN
