File: kicad/Ninja-qPCR/batch2/photosensing/qPCR-photosensing.sch (KiCad schematic (older format))
At the start: 27 parts, among them J1 Conn_01x14_Male, J2 Conn_01x02_Male, J3 Conn_01x05_Male, J4 Conn_01x05_Male, U1 AD630ARZ, U2 ADS1219IPWR, U3 LME49721MAX_NOPB

Commit message: sync
Parts:
- C1, C3, C7, C9: footprint Resistors_SMD:R_0603_HandSoldering -> Capacitors_SMD:C_0603_HandSoldering
- C11, C12, C6, C8: footprint Resistors_SMD:R_1206_HandSoldering -> Capacitors_SMD:C_1206_HandSoldering
- C2, C4, C5: value C -> 0.1uF?
Changed lines of the file:
@@
 F 0 "C12" H 10315 1346 50  0000 L CNN
 F 1 "0.22uF" H 10315 1255 50  0000 L CNN
-F 2 "Resistors_SMD:R_1206_HandSoldering" H 10238 1150 50  0001 C CNN
+F 2 "Capacitors_SMD:C_1206_HandSoldering" H 10238 1150 50  0001 C CNN
 F 3 "~" H 10200 1300 50  0001 C CNN
 	1    10200 1300
@@
 F 0 "C11" H 10015 1346 50  0000 L CNN
 F 1 "0.22uF" H 10015 1255 50  0000 L CNN
-F 2 "Resistors_SMD:R_1206_HandSoldering" H 9938 1150 50  0001 C CNN
+F 2 "Capacitors_SMD:C_1206_HandSoldering" H 9938 1150 50  0001 C CNN
 F 3 "~" H 9900 1300 50  0001 C CNN
 	1    9900 1300
@@
 F 0 "C9" H 9265 2696 50  0000 L CNN
 F 1 "0.1uF" H 9265 2605 50  0000 L CNN
-F 2 "Resistors_SMD:R_0603_HandSoldering" H 9188 2500 50  0001 C CNN
+F 2 "Capacitors_SMD:C_0603_HandSoldering" H 9188 2500 50  0001 C CNN
 F 3 "~" H 9150 2650 50  0001 C CNN
 	1    9150 2650
@@
 F 0 "C7" H 7215 3096 50  0000 L CNN
 F 1 "0.1uF" H 7215 3005 50  0000 L CNN
-F 2 "Resistors_SMD:R_0603_HandSoldering" H 7138 2900 50  0001 C CNN
+F 2 "Capacitors_SMD:C_0603_HandSoldering" H 7138 2900 50  0001 C CNN
 F 3 "~" H 7100 3050 50  0001 C CNN
 	1    7100 3050
@@
 F 0 "C3" H 2515 6846 50  0000 L CNN
 F 1 "0.1uF" H 2515 6755 50  0000 L CNN
-F 2 "Resistors_SMD:R_0603_HandSoldering" H 2438 6650 50  0001 C CNN
+F 2 "Capacitors_SMD:C_0603_HandSoldering" H 2438 6650 50  0001 C CNN
 F 3 "~" H 2400 6800 50  0001 C CNN
 	1    2400 6800
@@
 F 0 "C1" H 1615 6846 50  0000 L CNN
 F 1 "0.1uF" H 1615 6755 50  0000 L CNN
-F 2 "Resistors_SMD:R_0603_HandSoldering" H 1538 6650 50  0001 C CNN
+F 2 "Capacitors_SMD:C_0603_HandSoldering" H 1538 6650 50  0001 C CNN
 F 3 "~" H 1500 6800 50  0001 C CNN
 	1    1500 6800
@@
 F 0 "C6" H 6715 4546 50  0000 L CNN
 F 1 "0.47uF" H 6715 4455 50  0000 L CNN
-F 2 "Resistors_SMD:R_1206_HandSoldering" H 6638 4350 50  0001 C CNN
+F 2 "Capacitors_SMD:C_1206_HandSoldering" H 6638 4350 50  0001 C CNN
 F 3 "~" H 6600 4500 50  0001 C CNN
 	1    6600 4500
@@
 F 0 "C8" V 6948 4500 50  0000 C CNN
 F 1 "0.47uF" V 7039 4500 50  0000 C CNN
-F 2 "Resistors_SMD:R_1206_HandSoldering" H 7238 4350 50  0001 C CNN
+F 2 "Capacitors_SMD:C_1206_HandSoldering" H 7238 4350 50  0001 C CNN
 F 3 "~" H 7200 4500 50  0001 C CNN
 	1    7200 4500
@@
 P 2250 3750
 F 0 "C2" H 2365 3796 50  0000 L CNN
-F 1 "C" H 2365 3705 50  0000 L CNN
+F 1 "0.1uF?" H 2365 3705 50  0000 L CNN
 F 2 "Capacitors_SMD:C_0805_HandSoldering" H 2288 3600 50  0001 C CNN
 F 3 "~" H 2250 3750 50  0001 C CNN
@@
 P 3000 3750
 F 0 "C4" H 3115 3796 50  0000 L CNN
-F 1 "C" H 3115 3705 50  0000 L CNN
+F 1 "0.1uF?" H 3115 3705 50  0000 L CNN
 F 2 "Capacitors_SMD:C_0805_HandSoldering" H 3038 3600 50  0001 C CNN
 F 3 "~" H 3000 3750 50  0001 C CNN
@@
 P 4000 3750
 F 0 "C5" H 4115 3796 50  0000 L CNN
-F 1 "C" H 4115 3705 50  0000 L CNN
+F 1 "0.1uF?" H 4115 3705 50  0000 L CNN
 F 2 "Capacitors_SMD:C_0805_HandSoldering" H 4038 3600 50  0001 C CNN
 F 3 "~" H 4000 3750 50  0001 C CNN
