File: kicad/Ninja-qPCR/batch3/greengrass/greengrass.kicad_pcb (KiCad board)
At the start: 2 copper layers, 10 x 14 mm, 3 parts, among them J1 Conn_01x05_Male, J3 Conn_01x04_Male

Commit message: add batch3/gg. remove batch3/main
Changed lines of the file:
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@@
     (polygon
       (pts
-        (xy 133 79.5) (xy 120 79.5) (xy 120 63) (xy 133 63)
+        (xy 128.5 79.75) (xy 120 79.5) (xy 120 63) (xy 128.5 63.25)
       )
     )
@@
     (polygon
       (pts
-        (xy 132.5 79) (xy 120.5 79) (xy 120.5 63.5) (xy 132.5 63.5)
+        (xy 128.5 78.95) (xy 120.5 79) (xy 120.5 63.5) (xy 128.5 63.45)
       )
     )
