File: kicad/Ninja-qPCR/batch2/main/filePower.sch (KiCad schematic (older format))
At the start: 55 parts, among them J8 Barrel_Jack_Switch, J9 ATX-24, U1 DIN4_PWR, U2 IFX1763, U3 BD9D320EFJ-E2, U4 LTC3260EMSE-TRPBF, U5 CJT1117-3.3

Commit message: main wired
Parts:
- gave numbers to parts that had none: 1
- renumbered R21 to R22, R22 to R23, R23 to R24, R24 to R25, R25 to R26, R26 to R27, R27 to R28
Connections:
- net C-: now also U4.8 (NC)
- net at C24.1, U4.10 (C+): now also U4.9 (NC)

Commit message: sync
Parts:
- C23: footprint Capacitors_SMD:C_0603_HandSoldering -> Capacitors_SMD:C_0805_HandSoldering
- R21: value 100K -> 10K
- R24: value 120k -> 220k
- R25: value 1.8k/0 -> 0
- R26: value 22k -> 39k
Changed lines of the file:
@@
 P 8250 3050
 F 0 "R24" H 8320 3096 50  0000 L CNN
-F 1 "120k" H 8320 3005 50  0000 L CNN
+F 1 "220k" H 8320 3005 50  0000 L CNN
 F 2 "Resistors_SMD:R_0603_HandSoldering" V 8180 3050 50  0001 C CNN
 F 3 "~" H 8250 3050 50  0001 C CNN
@@
 P 8250 3850
 F 0 "R26" H 8320 3896 50  0000 L CNN
-F 1 "22k" H 8320 3805 50  0000 L CNN
+F 1 "39k" H 8320 3805 50  0000 L CNN
 F 2 "Resistors_SMD:R_0603_HandSoldering" V 8180 3850 50  0001 C CNN
 F 3 "~" H 8250 3850 50  0001 C CNN
@@
 P 8250 3400
 F 0 "R25" H 8320 3446 50  0000 L CNN
-F 1 "1.8k/0" H 8320 3355 50  0000 L CNN
+F 1 "0" H 8320 3355 50  0000 L CNN
 F 2 "Resistors_SMD:R_0603_HandSoldering" V 8180 3400 50  0001 C CNN
 F 3 "~" H 8250 3400 50  0001 C CNN
@@
 F 0 "C23" H 5465 5446 50  0000 L CNN
 F 1 "820pF" H 5465 5355 50  0000 L CNN
-F 2 "Capacitors_SMD:C_0603_HandSoldering" H 5388 5250 50  0001 C CNN
+F 2 "Capacitors_SMD:C_0805_HandSoldering" H 5388 5250 50  0001 C CNN
 F 3 "~" H 5350 5400 50  0001 C CNN
 	1    5350 5400
@@
 P 3750 2050
 F 0 "R21" H 3820 2096 50  0000 L CNN
-F 1 "100K" H 3820 2005 50  0000 L CNN
+F 1 "10K" H 3820 2005 50  0000 L CNN
 F 2 "Resistors_SMD:R_0603_HandSoldering" V 3680 2050 50  0001 C CNN
 F 3 "~" H 3750 2050 50  0001 C CNN
