File: kicad/Ninja-qPCR/batch9/outline/outline.kicad_pcb (KiCad board)
At the start: 2 copper layers, 100 x 120 mm, 7 parts, among them J1 Barrel_Jack_Switch, J2 Conn_01x40_Female

Commit message: batch9
Parts:
- moved C1 30.1 mm to (186.0, 89.0)
- moved C2 30.1 mm to (186.0, 102.5)
- moved C3 30.1 mm to (186.0, 116.0)
- moved C4 30.1 mm to (186.0, 143.0)
- moved C5 30.1 mm to (186.0, 129.5)
- moved J1 2.00 mm to (205.3, 97.0)
Other:
- board size 100 x 120 mm -> 96 x 116 mm
