File: kicad/Ninja-qPCR/batch11/breakouts/breakouts.kicad_pcb (KiCad board)
At the start: 2 copper layers, 176.5 x 33 mm, 24 parts, among them J1 Conn_01x04_Male, J10 Conn_01x12_Male, J11 Conn_01x06_Male, J12 Conn_01x06_Male, J13 Conn_01x05_Male, J14 Conn_01x06_Male, J15 Conn_01x06_Male, J2 Conn_01x05_Male, J3 Conn_01x05_Male, J4 Conn_01x04_Male, J5 Conn_01x10_Male, J6 Conn_01x10_Male, J7 Conn_01x08_Male, J8 Conn_01x08_Male, J9 Conn_01x12_Male, K1 EX2-2U1S, K2 EP2-3L3SAb, U1 A4955GLPTR-T, U2 AM4967, U3 BD61250MUV-E2‎, U4 8-PowerTDFN-PN, U5 8-PowerTDFN-NN, U6 SiZ346DT, U7 AOZ2264QI-19

Commit message: ordered batch11
Other:
- board text added: "AITENDO"
- board text added: "LATER"
- board text added: "ORDER"
- board text added: "USE PELTIER INSTEAD"
