File: kicad/Ninja-qPCR/batch13/peltier+relay/peltier+relay.kicad_pcb (KiCad board)
At the start: 2 copper layers, 79.7 x 32.7 mm, 33 parts, among them J1 Conn_01x02_Female, J2 Conn_01x03_Male, J3 Conn_01x02_Female, J4 Conn_01x02_Female, J5 Conn_01x05_Male, J6 Barrel_Jack_Switch, J7 Barrel_Jack_Switch, J8 Conn_01x03_Male, K1 EP2-3L3SAb, K2 EX2-2U1S, Q1 8-PowerVDFN-N, Q2 Q_NPN_BCE, Q4 Q_NPN_BCE, U1 AOZ2264QI-19, U2 MCP4551T-104

Commit message: update footprint
Parts:
- U1: footprint Ninja-qPCR:AOZ2264QI-19 -> Ninja-qPCR:AOZ2264QI-19-Long
- moved R3 1.37 mm to (165.2, 92.2)
Routing:
- net GND: track 187.0 -> 192.1 mm, vias 94 -> 93
- net REG_FB: track 26.3 -> 26.8 mm
Other:
- outline, holes or cut-outs redrawn
- board text added: "batch13/peltier+relay"
- board text removed: "batch12/peltier+relay"
