File: kicad/Ninja-qPCR/batch14/main/qPCR-main.kicad_pcb (KiCad board)
At the start: 2 copper layers, 100 x 100 mm, 141 parts, among them J1 Barrel_Jack_Switch, J10 Conn_01x01_Male, J11 Conn_01x01_Male, J12 Conn_01x01_Male, J13 Conn_01x01_Male, J14 Conn_01x01_Male, J15 Conn_01x01_Male, J16 Conn_01x01_Male, J17 Conn_01x02_Male, J18 Conn_01x60_Male, J19 Conn_01x01_Male, J2 Raspberry_Pi_3A_Plus_wpi, J20 Conn_01x01_Male, J3 Conn_01x01_Male, J4 Conn_01x01_Male, J5 Conn_01x01_Male, J6 Conn_01x01_Male, J7 Conn_01x01_Male, J8 Conn_01x01_Male, J9 Conn_01x01_Male, Q1 Q_NMOS_GSD, Q2 Q_NMOS_GSD, Q3 Q_NMOS_GSD, Q4 Q_NMOS_GSD, Q5 Q_NMOS_GSD, Q6 Q_NMOS_GSD, SW1 SW_Reed, U1 ADA2200ARUZ, U10 BD9D323QWZ-E2, U11 TL431DBZ, U12 TL431DBZ, U13 TL431DBZ, U14 TL431DBZ, U15 TL431DBZ, U16 CJT1117-3.3, U17 AP2210K-3.3TRG1, U18 SN74LVC1GU04DCKR, U19 CD74HC4067M96, U2 ADS122C04IPWR, U20 CD74HC4067M96, U21 TPS63710DRRR, U3 COM1305-0.032768-EXT-T-TR, U4 LMP7717MF_NOPB, U5 TS12A12511DCNR, U6 MCP4551T-503E/MS, U7 PCA9955B, U8 TS12A12511DCNR, U9 SN74LV4051APWR

Commit message: start batch14/main
Parts:
- removed J19, J20: Conn_01x01_Male, Pin_Headers:Pin_Header_Straight_1x01_Pitch2.54mm
- added C43: 10uF, Capacitors_SMD:C_0805, F.Cu at (170.5, 19.5)
- added C44: 0.1uF, Capacitors_SMD:C_0603, F.Cu at (155.3, 33.3)
- added C45: 1uF, Capacitors_SMD:C_0603, F.Cu at (159.8, 30.5)
- added C46: 22uF, Capacitors_SMD:C_1210, F.Cu at (150.6, 31.4)
- added C47: 0.1uF, Capacitors_SMD:C_0603, F.Cu at (169.3, 22.6)
- added C48: 1uF, Capacitors_SMD:C_0603, F.Cu at (174.8, 16.6)
- added C9: 10uF, Capacitors_SMD:C_0805, F.Cu at (155.6, 30.7)
- added D4: DIODE, Diodes_SMD:D_SMA, F.Cu at (145.8, 25.9)
- added D5: DIODE, Diodes_SMD:D_SMA, F.Cu at (172.2, 8.58)
- added HLID3: Screw_Terminal_01x02, Ninja-qPCR:TB_SeeedOPL_320110028, F.Cu at (155.9, 25.4)
- added K1: EP2-3L3SAb, Ninja-qPCR:EP2-3L3SAb, F.Cu at (130.5, 17.2)
- added K2: EX2-2U1S, Ninja-qPCR:EX2-2U1S, F.Cu at (157.2, 9.14)
- added L3: 3.3uH, Ninja-qPCR:104CDMCCDS-2R2MC, F.Cu at (134.4, 29.2)
- added Q7: Q_NPN_BCE, TO_SOT_Packages_SMD:SOT-23, F.Cu at (175.1, 13.1)
- added Q8: Q_NPN_BCE, TO_SOT_Packages_SMD:SOT-23, F.Cu at (164.4, 28.2)
- added R31: 10k, Resistors_SMD:R_0603, F.Cu at (174.5, 19.3)
- added R32: 60k, Resistors_SMD:R_0603, F.Cu at (159.7, 32.9)
- added R33: 5k, Resistors_SMD:R_0603, F.Cu at (163.5, 31.7)
- added R34: 10k, Resistors_SMD:R_0603, F.Cu at (173.0, 22.1)
- added U22: AOZ2264QI-19, Ninja-qPCR:AOZ2264QI-19-Long, F.Cu at (144.8, 31.2)
- added U23: MCP4551T-104, Ninja-qPCR:MCP4551T-104E&slash_MF, F.Cu at (164.8, 23.7)
- C16: footprint Capacitors_SMD:C_0603 -> Capacitors_SMD:C_0805
- J10: value Conn_01x01_Male -> Conn_01x02_Female; footprint Pin_Headers:Pin_Header_Straight_1x01_Pitch2.54mm -> Pin_Headers:Pin_Header_Straight_1x02_Pitch2.54mm
- U19, U20: footprint Ninja-qPCR:SOP65P780X200-24N -> Ninja-qPCR:CD74HC4067M96
- U6: footprint Ninja-qPCR:MCP4551T-502E&slash_MS -> Ninja-qPCR:MCP4551T-104E&slash_MF
- moved R16 140.8 mm to (209.1, 235.9), turned to 0 degrees
- moved C11 140.3 mm to (217.1, 219.1), turned to 270 degrees
- moved J18 139.8 mm to (215.1, 217.0)
- moved U18 138.8 mm to (208.9, 232.4)
- moved C10 138.2 mm to (213.7, 236.0), turned to 0 degrees
- moved U19 138.1 mm to (200.6, 227.0), turned to 0 degrees
- moved U20 137.9 mm to (188.6, 227.0), turned to 0 degrees
- moved U6 137.1 mm to (213.5, 232.4), turned to 270 degrees
- moved J10 136.6 mm to (170.5, 13.2), turned to 0 degrees
- moved U7 135.3 mm to (211.3, 223.9)
- moved C2 106.1 mm to (121.1, 227.6)
- moved C31 106.1 mm to (152.9, 232.1)
- moved C37 106.1 mm to (118.8, 222.1)
- moved C8 106.1 mm to (127.5, 223.1)
- moved JP1 106.1 mm to (136.1, 234.7)
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Connections:
- J10 pad 1: /GPIO28 -> REG_OUT
- J2 pad 37: /GPIO25 -> PEL_REG_EN
- J2 pad 38: /GPIO28 -> PEL_SWA
- J2 pad 40: /GPIO29 -> PEL_SWB
- U19 pad 16: /PhotoMUX/S_PD_OUT16 -> /PhotoMUX/S_PD_OUT9
- U19 pad 17: /PhotoMUX/S_PD_OUT15 -> /PhotoMUX/S_PD_OUT10
- U19 pad 18: /PhotoMUX/S_PD_OUT14 -> /PhotoMUX/S_PD_OUT11
- U19 pad 19: /PhotoMUX/S_PD_OUT13 -> /PhotoMUX/S_PD_OUT12
- U19 pad 20: /PhotoMUX/S_PD_OUT12 -> /PhotoMUX/S_PD_OUT13
- U19 pad 21: /PhotoMUX/S_PD_OUT11 -> /PhotoMUX/S_PD_OUT14
- U19 pad 22: /PhotoMUX/S_PD_OUT10 -> /PhotoMUX/S_PD_OUT15
- U19 pad 23: /PhotoMUX/S_PD_OUT9 -> /PhotoMUX/S_PD_OUT16
- U20 pad 16: /PhotoMUX/N_PD_OUT1 -> /PhotoMUX/N_PD_OUT8
- U20 pad 17: /PhotoMUX/N_PD_OUT2 -> /PhotoMUX/N_PD_OUT7
- U20 pad 18: /PhotoMUX/N_PD_OUT3 -> /PhotoMUX/N_PD_OUT6
- U20 pad 19: /PhotoMUX/N_PD_OUT4 -> /PhotoMUX/N_PD_OUT5
- U20 pad 20: /PhotoMUX/N_PD_OUT5 -> /PhotoMUX/N_PD_OUT4
- U20 pad 21: /PhotoMUX/N_PD_OUT6 -> /PhotoMUX/N_PD_OUT3
- U20 pad 22: /PhotoMUX/N_PD_OUT7 -> /PhotoMUX/N_PD_OUT2
- U20 pad 23: /PhotoMUX/N_PD_OUT8 -> /PhotoMUX/N_PD_OUT1
- U21 pad V: GND -> (no net)
- U7 pad 11: S_LED_OUT5 -> S_LED_OUT1
- U7 pad 12: S_LED_OUT6 -> S_LED_OUT2
- U7 pad 13: S_LED_OUT7 -> S_LED_OUT3
- U7 pad 14: S_LED_OUT8 -> S_LED_OUT4
- U7 pad 15: N_LED_OUT8 -> N_LED_OUT5
- U7 pad 16: N_LED_OUT7 -> N_LED_OUT6
- U7 pad 17: N_LED_OUT6 -> N_LED_OUT7
- U7 pad 18: N_LED_OUT5 -> N_LED_OUT8
- U7 pad 6: S_LED_OUT1 -> S_LED_OUT8
- U7 pad 7: S_LED_OUT2 -> S_LED_OUT7
- U7 pad 8: S_LED_OUT3 -> S_LED_OUT6
- U7 pad 9: S_LED_OUT4 -> S_LED_OUT5
Routing:
- net 3V3D: track 269.2 -> 227.3 mm, vias 10 -> 8
- net GNDA: track 216.0 -> 179.4 mm, vias 64 -> 38
- net 12V_UPS: track 67.1 -> 32.4 mm
- net PD_TH2: track 52.8 -> 18.2 mm, vias 2 -> 1
- net PD_TH1: track 51.7 -> 23.1 mm, vias 2 -> 1
- net THERM_EXT1: track 112.4 -> 90.7 mm
- net THERM_EXT3: track 117.9 -> 96.8 mm
- net 5V_UPS: track 173.6 -> 152.8 mm
- net THERM_EXT2: track 110.4 -> 89.7 mm
- net THERM_WELL: track 105.0 -> 85.1 mm
- net THERM_LID: track 108.6 -> 89.7 mm
- net THERM_AIR: track 105.0 -> 86.5 mm
- net PD_MUX_OUT: track 21.0 -> 6.31 mm
- net PEL_REG_EN: track 0.00 -> 13.4 mm
- net /GPIO25: track 13.4 -> 0.00 mm
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Other:
- net class Default: clearance 0.127 -> 0.1524; trace_width 0.127 -> 0.1524
- rule trace_clearance: 0.127 -> 0.1524

Commit message: wire
Parts:
- moved U8 81.0 mm to (215.1, 259.2)
- moved U9 80.0 mm to (221.4, 259.6)
- moved R18 79.7 mm to (213.6, 265.9)
- moved R17 77.6 mm to (213.4, 262.7)
- moved C1 73.7 mm to (194.9, 244.1), turned to 270 degrees
- moved R10 72.6 mm to (195.0, 241.0), turned to 90 degrees
- moved C4 67.7 mm to (199.9, 242.6), turned to 90 degrees
- moved C3 67.6 mm to (209.4, 242.6)
- moved U2 67.3 mm to (204.5, 242.6)
- moved C2 66.5 mm to (185.4, 244.3)
- moved J14 64.6 mm to (197.0, 243.2), turned to 90 degrees
- moved J15 64.6 mm to (197.0, 240.6), turned to 90 degrees
- moved U1 64.5 mm to (190.2, 242.9), turned to 0 degrees
- moved J16 61.4 mm to (183.5, 235.5)
- moved U3 55.0 mm to (184.7, 241.5), turned to 0 degrees
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Routing:
- net PD_MUX_OUT: track 6.31 -> 42.5 mm, vias 0 -> 2
- net GND: track 521.4 -> 489.0 mm, vias 309 -> 298
- net 3V3D: track 227.3 -> 245.0 mm, vias 8 -> 7
- net /Photo/PHOTO_OUT_N: track 14.5 -> 0.00 mm
- net /Photo/PHOTO_OUT_P: track 12.6 -> 0.00 mm
- net Net-(R16-Pad1): track 0.00 -> 11.4 mm, vias 0 -> 2
- net /Photo/GAIN_SMALL: track 6.33 -> 16.2 mm
- net /Photo/GAIN_LARGE: track 10.5 -> 19.6 mm
- net Net-(C2-Pad1): track 8.57 -> 0.00 mm, vias 2 -> 0
- net MUX_SELECT: track 73.5 -> 66.3 mm, vias 3 -> 2
- net /Photo/AMP_GAIN_SW: track 1.75 -> 8.73 mm
- net GNDA: track 179.4 -> 172.5 mm, vias 38 -> 17
- net Net-(R11-Pad1): track 5.87 -> 0.00 mm
- net Net-(C1-Pad1): track 4.74 -> 0.00 mm
- net CLKIN: track 3.64 -> 0.00 mm
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
Commit message: sync
Parts:
- added J19: Conn_01x24_Male, Ninja-qPCR:ATX24, B.Cu at (153.1, 41.5)
- J10: moved to B.Cu
- moved U9 156.0 mm to (134.1, 130.2)
- moved R18 155.3 mm to (128.4, 136.1), turned to 0 degrees
- moved U8 154.9 mm to (127.5, 131.4), turned to 180 degrees
- moved R17 154.3 mm to (125.2, 136.1), turned to 0 degrees
- moved J14 142.9 mm to (113.7, 127.0), turned to 270 degrees
- moved J15 139.3 mm to (116.3, 127.0), turned to 270 degrees
- moved R11 138.8 mm to (107.8, 128.0), turned to 180 degrees
- moved U2 138.7 mm to (121.6, 131.4)
- moved C3 137.9 mm to (121.8, 136.1), turned to 180 degrees
- moved C1 136.5 mm to (111.3, 136.1), turned to 180 degrees
- moved R10 136.4 mm to (107.8, 136.1), turned to 180 degrees
- moved U1 135.4 mm to (113.3, 131.4)
- moved C7 134.1 mm to (107.8, 129.8)
- moved C4 133.9 mm to (118.7, 136.1), turned to 0 degrees
- moved U3 133.9 mm to (107.8, 131.9)
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Connections:
- K2 pad 10: /SheetPeltier/PEL2 -> GND
- K2 pad 4: /SheetPeltier/PEL2 -> GND
Routing:
- net DOPEN: track 146.2 -> 0.00 mm, vias 2 -> 0
- net 12V: track 283.5 -> 147.9 mm, vias 3 -> 1
- net GND: track 489.0 -> 357.9 mm, vias 298 -> 79
- net VIN_SENSE: track 106.2 -> 0.45 mm, vias 4 -> 0
- net THERM_EXT3: track 96.8 -> 0.28 mm, vias 2 -> 0
- net THERM_EXT1: track 90.7 -> 0.00 mm, vias 2 -> 0
- net 3V3D: track 245.0 -> 154.8 mm, vias 7 -> 10
- net GNDA: track 172.5 -> 82.4 mm, vias 17 -> 11
- net THERM_LID: track 89.7 -> 0.00 mm, vias 2 -> 0
- net THERM_EXT2: track 89.7 -> 0.00 mm, vias 2 -> 0
- net /LID_HEATER: track 90.0 -> 1.66 mm, vias 2 -> 0
- net THERM_AIR: track 86.5 -> 0.00 mm, vias 2 -> 0
- net THERM_WELL: track 85.1 -> 0.28 mm, vias 2 -> 0
- net REG_OUT: track 0.00 -> 75.0 mm
- net /FAN: track 72.6 -> 1.66 mm, vias 1 -> 0
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- removed copper zone on B.Cu, net GNDA
- removed copper zone on F.Cu, net GNDA
Other:
- board size 100 x 100 mm -> 111.2 x 116 mm
- board text added: "batch14/main"
- board text removed: "25"
- board text removed: "28"
- board text removed: "29"
- board text removed: "batch10/main"
