File: kicad/Ninja-qPCR/batch18/5VUPS/5VUPS.kicad_sch (KiCad schematic)
At the start: 13 parts, among them U10 AP6503

Commit message: sync
Parts:
- removed C17: 22uF, Capacitor_SMD:C_1210_3225Metric, symbol Device:C
- C?: renamed from C12; footprint Capacitor_SMD:C_1210_3225Metric -> Capacitors_SMD:C_1210
- C?: renamed from C16; footprint Capacitor_SMD:C_1210_3225Metric -> Capacitors_SMD:C_1210
- C?: renamed from C13; footprint Capacitor_SMD:C_0603_1608Metric -> Capacitors_SMD:C_0603
- C?: renamed from C15; footprint Capacitor_SMD:C_0603_1608Metric -> Capacitors_SMD:C_0603
- C?: renamed from C14; footprint Capacitor_SMD:C_0603_1608Metric -> Capacitors_SMD:C_0603
- R?: renamed from R35; footprint Resistor_SMD:R_0603_1608Metric -> Resistors_SMD:R_0603
- R?: renamed from R37; footprint Resistor_SMD:R_0603_1608Metric -> Resistors_SMD:R_0603
- R?: renamed from R19; value 150k -> 100k/150k; footprint Resistor_SMD:R_0603_1608Metric -> Resistors_SMD:R_0603
- R?: renamed from R20; footprint Resistor_SMD:R_0603_1608Metric -> Resistors_SMD:R_0603
- R?: renamed from R36; footprint Resistor_SMD:R_0603_1608Metric -> Resistors_SMD:R_0603
- renumbered L1 to L?, U10 to U?
Other:
- note added: "Place one more 22uF for main in future"
Changed lines of the file:
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@@
     (stroke (width 0) (type default) (color 0 0 0 0))
+  )
+  (text "Place one more 22uF for main in future" (at 193.04 87.63 0)
+    (effects (font (size 1.27 1.27)) (justify left bottom))
   )
   (global_label "5V_UPS" (shape input) (at 198.12 77.47 0) (fields_autoplaced)
@@
   (symbol (lib_id "Device:L") (at 163.83 77.47 270) (mirror x) (unit 1)
     (in_bom yes) (on_board yes)
-    (property "Reference" "L1" (id 0) (at 163.83 72.644 90))
+    (property "Reference" "L?" (id 0) (at 163.83 72.644 90))
     (property "Value" "10uH" (id 1) (at 163.83 74.9554 90))
     (property "Footprint" "Ninja-qPCR:VLS6045EX-3R3N" (id 2) (at 163.83 77.47 0)
@@
   (symbol (lib_id "power:GND") (at 149.86 113.03 0) (mirror y) (unit 1)
     (in_bom yes) (on_board yes)
-    (property "Reference" "#PWR0108" (id 0) (at 149.86 119.38 0)
+    (property "Reference" "#PWR?" (id 0) (at 149.86 119.38 0)
       (effects (font (size 1.27 1.27)) hide)
     )
@@
   (symbol (lib_id "Device:R") (at 149.86 102.87 0) (mirror y) (unit 1)
     (in_bom yes) (on_board yes)
-    (property "Reference" "R35" (id 0) (at 148.082 101.7016 0)
+    (property "Reference" "R?" (id 0) (at 148.082 101.7016 0)
       (effects (font (size 1.27 1.27)) (justify left))
     )
@@
       (effects (font (size 1.27 1.27)) (justify left))
     )
-    (property "Footprint" "Resistor_SMD:R_0603_1608Metric" (id 2) (at 151.638 102.87 90)
+    (property "Footprint" "Resistors_SMD:R_0603" (id 2) (at 151.638 102.87 90)
       (effects (font (size 1.27 1.27)) hide)
     )
@@
     (pin "2")
   )
-  (symbol (lib_id "Device:C") (at 194.31 87.63 0) (mirror x) (unit 1)
-    (in_bom yes) (on_board yes)
-    (property "Reference" "C17" (id 0) (at 191.389 86.4616 0)
-      (effects (font (size 1.27 1.27)) (justify right))
-    )
-    (property "Value" "22uF" (id 1) (at 191.389 88.773 0)
-      (effects (font (size 1.27 1.27)) (justify right))
-    )
-    (property "Footprint" "Capacitor_SMD:C_1210_3225Metric" (id 2) (at 195.2752 83.82 0)
-      (effects (font (size 1.27 1.27)) hide)
-    )
-    (property "Datasheet" "~" (id 3) (at 194.31 87.63 0)
-      (effects (font (size 1.27 1.27)) hide)
-    )
-    (pin "1")
-    (pin "2")
-  )
   (symbol (lib_id "power:GND") (at 105.41 92.71 0) (unit 1)
     (in_bom yes) (on_board yes)
-    (property "Reference" "#PWR0104" (id 0) (at 105.41 99.06 0)
+    (property "Reference" "#PWR?" (id 0) (at 105.41 99.06 0)
       (effects (font (size 1.27 1.27)) hide)
     )
@@
   (symbol (lib_id "Device:C") (at 105.41 86.36 0) (mirror x) (unit 1)
     (in_bom yes) (on_board yes)
-    (property "Reference" "C12" (id 0) (at 102.489 85.1916 0)
+    (property "Reference" "C?" (id 0) (at 102.489 85.1916 0)
       (effects (font (size 1.27 1.27)) (justify right))
     )
@@
       (effects (font (size 1.27 1.27)) (justify right))
     )
-    (property "Footprint" "Capacitor_SMD:C_1210_3225Metric" (id 2) (at 106.3752 82.55 0)
+    (property "Footprint" "Capacitors_SMD:C_1210" (id 2) (at 106.3752 82.55 0)
       (effects (font (size 1.27 1.27)) hide)
     )
@@
   (symbol (lib_id "power:GND") (at 194.31 93.98 0) (mirror y) (unit 1)
     (in_bom yes) (on_board yes)
-    (property "Reference" "#PWR0113" (id 0) (at 194.31 100.33 0)
+    (property "Reference" "#PWR?" (id 0) (at 194.31 100.33 0)
       (effects (font (size 1.27 1.27)) hide)
     )
@@
   (symbol (lib_id "power:GND") (at 170.18 113.03 0) (mirror y) (unit 1)
     (in_bom yes) (on_board yes)
-    (property "Reference" "#PWR0107" (id 0) (at 170.18 119.38 0)
+    (property "Reference" "#PWR?" (id 0) (at 170.18 119.38 0)
       (effects (font (size 1.27 1.27)) hide)
     )
@@
   (symbol (lib_id "power:GND") (at 119.38 92.71 0) (unit 1)
     (in_bom yes) (on_board yes)
-    (property "Reference" "#PWR0105" (id 0) (at 119.38 99.06 0)
+    (property "Reference" "#PWR?" (id 0) (at 119.38 99.06 0)
       (effects (font (size 1.27 1.27)) hide)
     )
@@
   (symbol (lib_id "Device:R") (at 170.18 106.68 0) (mirror y) (unit 1)
     (in_bom yes) (on_board yes)
-    (property "Reference" "R37" (id 0) (at 168.402 105.5116 0)
+    (property "Reference" "R?" (id 0) (at 168.402 105.5116 0)
       (effects (font (size 1.27 1.27)) (justify left))
     )
@@
       (effects (font (size 1.27 1.27)) (justify left))
     )
-    (property "Footprint" "Resistor_SMD:R_0603_1608Metric" (id 2) (at 171.958 106.68 90)
+    (property "Footprint" "Resistors_SMD:R_0603" (id 2) (at 171.958 106.68 90)
       (effects (font (size 1.27 1.27)) hide)
     )
@@
   (symbol (lib_id "Device:C") (at 186.69 87.63 0) (mirror x) (unit 1)
     (in_bom yes) (on_board yes)
-    (property "Reference" "C16" (id 0) (at 183.769 86.4616 0)
+    (property "Reference" "C?" (id 0) (at 183.769 86.4616 0)
       (effects (font (size 1.27 1.27)) (justify right))
     )
@@
       (effects (font (size 1.27 1.27)) (justify right))
     )
-    (property "Footprint" "Capacitor_SMD:C_1210_3225Metric" (id 2) (at 187.6552 83.82 0)
+    (property "Footprint" "Capacitors_SMD:C_1210" (id 2) (at 187.6552 83.82 0)
       (effects (font (size 1.27 1.27)) hide)
     )
@@
   (symbol (lib_id "Device:R") (at 114.3 77.47 90) (mirror x) (unit 1)
     (in_bom yes) (on_board yes)
-    (property "Reference" "R19" (id 0) (at 113.1316 79.248 0)
-      (effects (font (size 1.27 1.27)) (justify left))
-    )
-    (property "Value" "150k" (id 1) (at 115.443 79.248 0)
-      (effects (font (size 1.27 1.27)) (justify left))
-    )
-    (property "Footprint" "Resistor_SMD:R_0603_1608Metric" (id 2) (at 114.3 75.692 90)
+    (property "Reference" "R?" (id 0) (at 113.1316 79.248 0)
+      (effects (font (size 1.27 1.27)) (justify left))
+    )
+    (property "Value" "100k/150k" (id 1) (at 115.443 79.248 0)
+      (effects (font (size 1.27 1.27)) (justify left))
+    )
+    (property "Footprint" "Resistors_SMD:R_0603" (id 2) (at 114.3 75.692 90)
       (effects (font (size 1.27 1.27)) hide)
     )
@@
   (symbol (lib_id "Device:R") (at 143.51 102.87 0) (mirror y) (unit 1)
     (in_bom yes) (on_board yes)
-    (property "Reference" "R20" (id 0) (at 141.732 101.7016 0)
+    (property "Reference" "R?" (id 0) (at 141.732 101.7016 0)
       (effects (font (size 1.27 1.27)) (justify left))
     )
@@
       (effects (font (size 1.27 1.27)) (justify left))
     )
-    (property "Footprint" "Resistor_SMD:R_0603_1608Metric" (id 2) (at 145.288 102.87 90)
+    (property "Footprint" "Resistors_SMD:R_0603" (id 2) (at 145.288 102.87 90)
       (effects (font (size 1.27 1.27)) hide)
     )
@@
   (symbol (lib_id "Device:C") (at 119.38 86.36 180) (unit 1)
     (in_bom yes) (on_board yes)
-    (property "Reference" "C13" (id 0) (at 114.3 86.36 0)
+    (property "Reference" "C?" (id 0) (at 114.3 86.36 0)
       (effects (font (size 1.27 1.27)) (justify right))
     )
@@
       (effects (font (size 1.27 1.27)) (justify right))
     )
-    (property "Footprint" "Capacitor_SMD:C_0603_1608Metric" (id 2) (at 118.4148 82.55 0)
+    (property "Footprint" "Capacitors_SMD:C_0603" (id 2) (at 118.4148 82.55 0)
       (effects (font (size 1.27 1.27)) hide)
     )
@@
   (symbol (lib_id "Device:R") (at 170.18 93.98 0) (mirror y) (unit 1)
     (in_bom yes) (on_board yes)
-    (property "Reference" "R36" (id 0) (at 168.402 92.8116 0)
+    (property "Reference" "R?" (id 0) (at 168.402 92.8116 0)
       (effects (font (size 1.27 1.27)) (justify left))
     )
@@
       (effects (font (size 1.27 1.27)) (justify left))
     )
-    (property "Footprint" "Resistor_SMD:R_0603_1608Metric" (id 2) (at 171.958 93.98 90)
+    (property "Footprint" "Resistors_SMD:R_0603" (id 2) (at 171.958 93.98 90)
       (effects (font (size 1.27 1.27)) hide)
     )
@@
   (symbol (lib_id "power:GND") (at 186.69 93.98 0) (mirror y) (unit 1)
     (in_bom yes) (on_board yes)
-    (property "Reference" "#PWR0114" (id 0) (at 186.69 100.33 0)
+    (property "Reference" "#PWR?" (id 0) (at 186.69 100.33 0)
       (effects (font (size 1.27 1.27)) hide)
     )
@@
   (symbol (lib_id "Device:C") (at 151.13 74.93 90) (unit 1)
     (in_bom yes) (on_board yes)
-    (property "Reference" "C15" (id 0) (at 151.13 69.85 0)
+    (property "Reference" "C?" (id 0) (at 151.13 69.85 0)
       (effects (font (size 1.27 1.27)) (justify right))
     )
@@
       (effects (font (size 1.27 1.27)) (justify right))
     )
-    (property "Footprint" "Capacitor_SMD:C_0603_1608Metric" (id 2) (at 154.94 73.9648 0)
+    (property "Footprint" "Capacitors_SMD:C_0603" (id 2) (at 154.94 73.9648 0)
       (effects (font (size 1.27 1.27)) hide)
     )
@@
   (symbol (lib_id "Device:C") (at 149.86 90.17 0) (mirror x) (unit 1)
     (in_bom yes) (on_board yes)
-    (property "Reference" "C14" (id 0) (at 146.939 89.0016 0)
+    (property "Reference" "C?" (id 0) (at 146.939 89.0016 0)
       (effects (font (size 1.27 1.27)) (justify right))
     )
@@
       (effects (font (size 1.27 1.27)) (justify right))
     )
-    (property "Footprint" "Capacitor_SMD:C_0603_1608Metric" (id 2) (at 150.8252 86.36 0)
+    (property "Footprint" "Capacitors_SMD:C_0603" (id 2) (at 150.8252 86.36 0)
       (effects (font (size 1.27 1.27)) hide)
     )
@@
   (symbol (lib_id "Ninja-qPCR:AP6503") (at 135.89 78.74 0) (unit 1)
     (in_bom yes) (on_board yes)
-    (property "Reference" "U10" (id 0) (at 135.89 69.215 0))
+    (property "Reference" "U?" (id 0) (at 135.89 69.215 0))
     (property "Value" "AP6503" (id 1) (at 135.89 71.5264 0))
     (property "Footprint" "Ninja-qPCR:AP6503" (id 2) (at 135.89 78.74 0)
@@
   (symbol (lib_id "power:GND") (at 125.73 92.71 0) (unit 1)
     (in_bom yes) (on_board yes)
-    (property "Reference" "#PWR0106" (id 0) (at 125.73 99.06 0)
-      (effects (font (size 1.27 1.27)) hide)
-    )
+    (property "Reference" "#PWR?" (id 0) (at 125.73 99.06 0)
+      (effects (font (size 1.27 1.27)) hide)
+    )
