File: kicad/Ninja-qPCR/batch18/main/file12V_UPS.kicad_sch (KiCad schematic)
At the start: 25 parts, among them J17 Conn_01x02_Male, U11 TL431DBZ, U12 TL431DBZ, U13 TL431DBZ, U14 TL431DBZ, U15 TL431DBZ

Commit message: replace chips
Parts:
- R21, R22: footprint Resistors_SMD:R_0603 -> Resistor_SMD:R_0603_1608Metric
- R24, R25, R26, R27, R28: footprint Resistors_SMD:R_2512 -> Resistor_SMD:R_2512_6332Metric
Changed lines of the file:
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@@
       (effects (font (size 1.27 1.27)) (justify left))
     )
-    (property "Footprint" "Resistors_SMD:R_0603" (id 2) (at 98.552 74.93 90)
+    (property "Footprint" "Resistor_SMD:R_0603_1608Metric" (id 2) (at 98.552 74.93 90)
       (effects (font (size 1.27 1.27)) hide)
     )
@@
       (effects (font (size 1.27 1.27)) (justify left))
     )
-    (property "Footprint" "Resistors_SMD:R_0603" (id 2) (at 98.552 64.77 90)
+    (property "Footprint" "Resistor_SMD:R_0603_1608Metric" (id 2) (at 98.552 64.77 90)
       (effects (font (size 1.27 1.27)) hide)
     )
@@
       (effects (font (size 1.27 1.27)) (justify right))
     )
-    (property "Footprint" "Resistors_SMD:R_2512" (id 2) (at 145.288 147.32 90)
+    (property "Footprint" "Resistor_SMD:R_2512_6332Metric" (id 2) (at 145.288 147.32 90)
       (effects (font (size 1.27 1.27)) hide)
     )
@@
       (effects (font (size 1.27 1.27)) (justify right))
     )
-    (property "Footprint" "Resistors_SMD:R_2512" (id 2) (at 145.288 130.81 90)
+    (property "Footprint" "Resistor_SMD:R_2512_6332Metric" (id 2) (at 145.288 130.81 90)
       (effects (font (size 1.27 1.27)) hide)
     )
@@
       (effects (font (size 1.27 1.27)) (justify right))
     )
-    (property "Footprint" "Resistors_SMD:R_2512" (id 2) (at 145.288 114.3 90)
+    (property "Footprint" "Resistor_SMD:R_2512_6332Metric" (id 2) (at 145.288 114.3 90)
       (effects (font (size 1.27 1.27)) hide)
     )
@@
       (effects (font (size 1.27 1.27)) (justify right))
     )
-    (property "Footprint" "Resistors_SMD:R_2512" (id 2) (at 145.288 97.79 90)
+    (property "Footprint" "Resistor_SMD:R_2512_6332Metric" (id 2) (at 145.288 97.79 90)
       (effects (font (size 1.27 1.27)) hide)
     )
@@
       (effects (font (size 1.27 1.27)) (justify right))
     )
-    (property "Footprint" "Resistors_SMD:R_2512" (id 2) (at 145.288 81.28 90)
-      (effects (font (size 1.27 1.27)) hide)
-    )
+    (property "Footprint" "Resistor_SMD:R_2512_6332Metric" (id 2) (at 145.288 81.28 90)
+      (effects (font (size 1.27 1.27)) hide)
+    )

Commit message: sync
Parts:
- J17: footprint Pin_Headers:Pin_Header_Straight_1x02_Pitch2.54mm -> Connector_PinHeader_2.54mm:PinHeader_1x02_P2.54mm_Vertical
- U11, U12, U13, U14: footprint TO_SOT_Packages_SMD:SOT-23 -> Package_TO_SOT_SMD:SOT-23
- U15: footprint TO_SOT_Packages_SMD:SOT-23 -> Package_TO_SOT_SMD:SOT-223
Changed lines of the file:
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@@
       (effects (font (size 1.27 1.27)) (justify right))
     )
-    (property "Footprint" "Pin_Headers:Pin_Header_Straight_1x02_Pitch2.54mm" (id 2) (at 182.88 64.77 0)
+    (property "Footprint" "Connector_PinHeader_2.54mm:PinHeader_1x02_P2.54mm_Vertical" (id 2) (at 182.88 64.77 0)
       (effects (font (size 1.27 1.27)) hide)
     )
@@
       (effects (font (size 1.27 1.27)) (justify right))
     )
-    (property "Footprint" "TO_SOT_Packages_SMD:SOT-23" (id 2) (at 115.57 81.28 0)
+    (property "Footprint" "Package_TO_SOT_SMD:SOT-23" (id 2) (at 115.57 81.28 0)
       (effects (font (size 1.27 1.27) italic) hide)
     )
@@
       (effects (font (size 1.27 1.27)) (justify right))
     )
-    (property "Footprint" "TO_SOT_Packages_SMD:SOT-23" (id 2) (at 115.57 97.79 0)
+    (property "Footprint" "Package_TO_SOT_SMD:SOT-23" (id 2) (at 115.57 97.79 0)
       (effects (font (size 1.27 1.27) italic) hide)
     )
@@
       (effects (font (size 1.27 1.27)) (justify right))
     )
-    (property "Footprint" "TO_SOT_Packages_SMD:SOT-23" (id 2) (at 115.57 114.3 0)
+    (property "Footprint" "Package_TO_SOT_SMD:SOT-23" (id 2) (at 115.57 114.3 0)
       (effects (font (size 1.27 1.27) italic) hide)
     )
@@
       (effects (font (size 1.27 1.27)) (justify right))
     )
-    (property "Footprint" "TO_SOT_Packages_SMD:SOT-23" (id 2) (at 115.57 130.81 0)
+    (property "Footprint" "Package_TO_SOT_SMD:SOT-23" (id 2) (at 115.57 130.81 0)
       (effects (font (size 1.27 1.27) italic) hide)
     )
@@
       (effects (font (size 1.27 1.27)) (justify right))
     )
-    (property "Footprint" "TO_SOT_Packages_SMD:SOT-23" (id 2) (at 115.57 147.32 0)
-      (effects (font (size 1.27 1.27) italic) hide)
-    )
+    (property "Footprint" "Package_TO_SOT_SMD:SOT-223" (id 2) (at 115.57 147.32 0)
+      (effects (font (size 1.27 1.27) italic) hide)
+    )

Commit message: wire
Parts:
- removed JP2, JP3: Jumper, Jumper:SolderJumper-2_P1.3mm_Open_TrianglePad1.0x1.5mm, symbol Device:Jumper
- added JP2: Jumper_3_Open, Jumper:SolderJumper-3_P2.0mm_Open_TrianglePad1.0x1.5mm, symbol Jumper:Jumper_3_Open
- U15: footprint Package_TO_SOT_SMD:SOT-223 -> Package_TO_SOT_SMD:SOT-23
Connections:
- net 12V: now also JP2.1 (A)
- net 12V_UPS: now also JP2.2 (C)
- net at D2.1 (K), D3.1 (K), F1.2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: now also JP2.3 (B)
Changed lines of the file:
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@@
+    (stroke (width 0) (type default) (color 0 0 0 0))
+  )
+  (wire (pts (xy 158.75 80.01) (xy 158.75 83.82))
     (stroke (width 0) (type default) (color 0 0 0 0))
   )
@@
     (stroke (width 0) (type default) (color 0 0 0 0))
   )
+  (wire (pts (xy 162.56 73.66) (xy 173.99 73.66))
+    (stroke (width 0) (type default) (color 0 0 0 0))
+  )
   (wire (pts (xy 121.92 81.28) (xy 124.46 81.28))
     (stroke (width 0) (type default) (color 0 0 0 0))
@@
     (stroke (width 0) (type default) (color 0 0 0 0))
   )
-  (wire (pts (xy 187.96 96.52) (xy 190.5 96.52))
-    (stroke (width 0) (type default) (color 0 0 0 0))
-  )
   (wire (pts (xy 119.38 137.16) (xy 129.54 137.16))
     (stroke (width 0) (type default) (color 0 0 0 0))
@@
     (stroke (width 0) (type default) (color 0 0 0 0))
   )
-  (wire (pts (xy 170.18 96.52) (xy 172.72 96.52))
-    (stroke (width 0) (type default) (color 0 0 0 0))
-  )
   (wire (pts (xy 124.46 97.79) (xy 124.46 90.17))
     (stroke (width 0) (type default) (color 0 0 0 0))
@@
     (stroke (width 0) (type default) (color 0 0 0 0))
   )
-  (wire (pts (xy 173.99 58.42) (xy 173.99 67.31))
+  (wire (pts (xy 173.99 58.42) (xy 173.99 73.66))
     (stroke (width 0) (type default) (color 0 0 0 0))
   )
@@
   )
   (wire (pts (xy 129.54 60.96) (xy 129.54 58.42))
+    (stroke (width 0) (type default) (color 0 0 0 0))
+  )
+  (wire (pts (xy 156.845 83.82) (xy 158.75 83.82))
     (stroke (width 0) (type default) (color 0 0 0 0))
   )
@@
     )
   )
-  (global_label "12V" (shape input) (at 170.18 96.52 180) (fields_autoplaced)
+  (global_label "12V" (shape input) (at 156.845 83.82 180) (fields_autoplaced)
     (effects (font (size 1.27 1.27)) (justify right))
-    (property "Intersheet References" "${INTERSHEET_REFS}" (id 0) (at 0 0 0)
-      (effects (font (size 1.27 1.27)) hide)
-    )
-  )
-  (global_label "12V_UPS" (shape input) (at 190.5 96.52 0) (fields_autoplaced)
-    (effects (font (size 1.27 1.27)) (justify left))
-    (property "Intersheet References" "${INTERSHEET_REFS}" (id 0) (at 0 0 0)
+    (property "Intersheet References" "${INTERSHEET_REFS}" (id 0) (at -13.335 -12.7 0)
       (effects (font (size 1.27 1.27)) hide)
     )
@@
     (pin "2")
   )
-  (symbol (lib_id "Device:Jumper") (at 166.37 67.31 0) (unit 1)
-    (in_bom yes) (on_board yes)
-    (property "Reference" "JP2" (id 0) (at 166.37 60.6044 0))
-    (property "Value" "Jumper" (id 1) (at 166.37 62.9158 0))
-    (property "Footprint" "Jumper:SolderJumper-2_P1.3mm_Open_TrianglePad1.0x1.5mm" (id 2) (at 166.37 67.31 0)
-      (effects (font (size 1.27 1.27)) hide)
-    )
-    (property "Datasheet" "~" (id 3) (at 166.37 67.31 0)
-      (effects (font (size 1.27 1.27)) hide)
-    )
-    (pin "1")
-    (pin "2")
-  )
   (symbol (lib_id "Device:R") (at 143.51 147.32 180) (unit 1)
     (in_bom yes) (on_board yes)
@@
     (pin "2")
   )
-  (symbol (lib_id "Device:Jumper") (at 180.34 96.52 0) (unit 1)
-    (in_bom yes) (on_board yes)
-    (property "Reference" "JP3" (id 0) (at 180.34 89.8144 0))
-    (property "Value" "Jumper" (id 1) (at 180.34 92.1258 0))
-    (property "Footprint" "Jumper:SolderJumper-2_P1.3mm_Open_TrianglePad1.0x1.5mm" (id 2) (at 180.34 96.52 0)
-      (effects (font (size 1.27 1.27)) hide)
-    )
-    (property "Datasheet" "~" (id 3) (at 180.34 96.52 0)
-      (effects (font (size 1.27 1.27)) hide)
-    )
-    (pin "1")
-    (pin "2")
-  )
   (symbol (lib_id "Reference_Voltage:TL431DBZ") (at 119.38 81.28 270) (mirror x) (unit 1)
     (in_bom yes) (on_board yes)
@@
       (effects (font (size 1.27 1.27)) (justify right))
     )
-    (property "Footprint" "Package_TO_SOT_SMD:SOT-223" (id 2) (at 115.57 147.32 0)
+    (property "Footprint" "Package_TO_SOT_SMD:SOT-23" (id 2) (at 115.57 147.32 0)
       (effects (font (size 1.27 1.27) italic) hide)
     )
@@
     )
     (pin "1")
+    (pin "2")
+    (pin "3")
+  )
+  (symbol (lib_id "Jumper:Jumper_3_Open") (at 158.75 73.66 90) (unit 1)
+    (in_bom yes) (on_board yes) (fields_autoplaced)
+    (property "Reference" "JP2" (id 0) (at 156.6159 72.7515 90)
+      (effects (font (size 1.27 1.27)) (justify left))
+    )
+    (property "Value" "Jumper_3_Open" (id 1) (at 156.6159 75.5266 90)
+      (effects (font (size 1.27 1.27)) (justify left))
+    )
+    (property "Footprint" "Jumper:SolderJumper-3_P2.0mm_Open_TrianglePad1.0x1.5mm" (id 2) (at 158.75 73.66 0)
+      (effects (font (size 1.27 1.27)) hide)
+    )
+    (property "Datasheet" "~" (id 3) (at 158.75 73.66 0)
+      (effects (font (size 1.27 1.27)) hide)
+    )
+    (pin "1")

Commit message: wired
Parts:
- J17: footprint Connector_PinHeader_2.54mm:PinHeader_1x02_P2.54mm_Vertical -> Connector_PinSocket_2.54mm:PinSocket_1x02_P2.54mm_Vertical
Changed lines of the file:
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@@
       (effects (font (size 1.27 1.27)) (justify right))
     )
-    (property "Footprint" "Connector_PinHeader_2.54mm:PinHeader_1x02_P2.54mm_Vertical" (id 2) (at 182.88 64.77 0)
+    (property "Footprint" "Connector_PinSocket_2.54mm:PinSocket_1x02_P2.54mm_Vertical" (id 2) (at 182.88 64.77 0)
       (effects (font (size 1.27 1.27)) hide)
     )
