File: kicad/Ninja-qPCR/batch18/main/filePeltier.kicad_sch (KiCad schematic)
At the start: 17 parts, among them J10 Conn_01x02_Male, K1 EP2-3L3SAb, K2 EX2-2U1S, Q7 Q_NPN_BCE, Q8 Q_NPN_BCE, Q9 SIRA88BDP-T1-GE3

Commit message: replace chips
Parts:
- C43, C9: footprint Capacitors_SMD:C_1210 -> Capacitor_SMD:C_1210_3225Metric
- R31, R32, R33, R34: footprint Resistors_SMD:R_0603 -> Resistor_SMD:R_0603_1608Metric
Changed lines of the file:
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@@
     (property "Reference" "R34" (id 0) (at 182.88 103.9622 90))
     (property "Value" "10k" (id 1) (at 182.88 106.2736 90))
-    (property "Footprint" "Resistors_SMD:R_0603" (id 2) (at 182.88 107.442 90)
+    (property "Footprint" "Resistor_SMD:R_0603_1608Metric" (id 2) (at 182.88 107.442 90)
       (effects (font (size 1.27 1.27)) hide)
     )
@@
     (property "Reference" "R31" (id 0) (at 116.84 103.9622 90))
     (property "Value" "10k" (id 1) (at 116.84 106.2736 90))
-    (property "Footprint" "Resistors_SMD:R_0603" (id 2) (at 116.84 107.442 90)
+    (property "Footprint" "Resistor_SMD:R_0603_1608Metric" (id 2) (at 116.84 107.442 90)
       (effects (font (size 1.27 1.27)) hide)
     )
@@
       (effects (font (size 1.27 1.27)) (justify left))
     )
-    (property "Footprint" "Resistors_SMD:R_0603" (id 2) (at 50.292 107.95 90)
+    (property "Footprint" "Resistor_SMD:R_0603_1608Metric" (id 2) (at 50.292 107.95 90)
       (effects (font (size 1.27 1.27)) hide)
     )
@@
       (effects (font (size 1.27 1.27)) (justify left))
     )
-    (property "Footprint" "Capacitors_SMD:C_1210" (id 2) (at 51.7652 81.28 0)
+    (property "Footprint" "Capacitor_SMD:C_1210_3225Metric" (id 2) (at 51.7652 81.28 0)
       (effects (font (size 1.27 1.27)) hide)
     )
@@
       (effects (font (size 1.27 1.27)) (justify left))
     )
-    (property "Footprint" "Capacitors_SMD:C_1210" (id 2) (at 87.3252 81.28 0)
+    (property "Footprint" "Capacitor_SMD:C_1210_3225Metric" (id 2) (at 87.3252 81.28 0)
       (effects (font (size 1.27 1.27)) hide)
     )
@@
       (effects (font (size 1.27 1.27)) (justify left))
     )
-    (property "Footprint" "Resistors_SMD:R_0603" (id 2) (at 41.91 99.822 90)
-      (effects (font (size 1.27 1.27)) hide)
-    )
+    (property "Footprint" "Resistor_SMD:R_0603_1608Metric" (id 2) (at 41.91 99.822 90)
+      (effects (font (size 1.27 1.27)) hide)
+    )

Commit message: sync
Parts:
- J10: footprint Pin_Headers:Pin_Header_Straight_1x02_Pitch2.54mm -> Connector_PinHeader_2.54mm:PinHeader_1x02_P2.54mm_Vertical
- Q7, Q8: footprint TO_SOT_Packages_SMD:SOT-23 -> Package_TO_SOT_SMD:SOT-23
Changed lines of the file:
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@@
       (effects (font (size 1.27 1.27)) (justify left))
     )
-    (property "Footprint" "TO_SOT_Packages_SMD:SOT-23" (id 2) (at 134.62 106.68 0)
+    (property "Footprint" "Package_TO_SOT_SMD:SOT-23" (id 2) (at 134.62 106.68 0)
       (effects (font (size 1.27 1.27)) hide)
     )
@@
       (effects (font (size 1.27 1.27)) (justify left))
     )
-    (property "Footprint" "TO_SOT_Packages_SMD:SOT-23" (id 2) (at 165.1 106.68 0)
+    (property "Footprint" "Package_TO_SOT_SMD:SOT-23" (id 2) (at 165.1 106.68 0)
       (effects (font (size 1.27 1.27)) hide)
     )
@@
     (property "Reference" "J10" (id 0) (at 119.5832 53.8226 0))
     (property "Value" "Conn_01x02_Male" (id 1) (at 119.5832 56.134 0))
-    (property "Footprint" "Pin_Headers:Pin_Header_Straight_1x02_Pitch2.54mm" (id 2) (at 116.84 58.42 0)
-      (effects (font (size 1.27 1.27)) hide)
-    )
+    (property "Footprint" "Connector_PinHeader_2.54mm:PinHeader_1x02_P2.54mm_Vertical" (id 2) (at 116.84 58.42 0)
+      (effects (font (size 1.27 1.27)) hide)
+    )

Commit message: wire
Parts:
- removed J10: Conn_01x02_Male, Connector_PinHeader_2.54mm:PinHeader_1x02_P2.54mm_Vertical, symbol Connector:Conn_01x02_Male
Changed lines of the file:
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@@
-    (stroke (width 0) (type default) (color 0 0 0 0))
-  )
-  (wire (pts (xy 121.92 60.96) (xy 127 60.96))
     (stroke (width 0) (type default) (color 0 0 0 0))
   )
@@
   )
   (wire (pts (xy 179.07 109.22) (xy 175.26 109.22))
-    (stroke (width 0) (type default) (color 0 0 0 0))
-  )
-  (wire (pts (xy 127 58.42) (xy 121.92 58.42))
     (stroke (width 0) (type default) (color 0 0 0 0))
   )
@@
     )
   )
-  (global_label "12V" (shape input) (at 127 58.42 0) (fields_autoplaced)
-    (effects (font (size 1.27 1.27)) (justify left))
-    (property "Intersheet References" "${INTERSHEET_REFS}" (id 0) (at 0 0 0)
-      (effects (font (size 1.27 1.27)) hide)
-    )
-  )
   (global_label "REG_OUT" (shape input) (at 88.9 86.36 0) (fields_autoplaced)
     (effects (font (size 1.27 1.27)) (justify left))
@@
   (global_label "12V" (shape input) (at 129.54 80.01 180) (fields_autoplaced)
     (effects (font (size 1.27 1.27)) (justify right))
-    (property "Intersheet References" "${INTERSHEET_REFS}" (id 0) (at 0 0 0)
-      (effects (font (size 1.27 1.27)) hide)
-    )
-  )
-  (global_label "REG_OUT" (shape input) (at 127 60.96 0) (fields_autoplaced)
-    (effects (font (size 1.27 1.27)) (justify left))
     (property "Intersheet References" "${INTERSHEET_REFS}" (id 0) (at 0 0 0)
       (effects (font (size 1.27 1.27)) hide)
@@
       (effects (font (size 1.27 1.27)) hide)
     )
-    (pin "1")
-    (pin "2")
-  )
-  (symbol (lib_id "Connector:Conn_01x02_Male") (at 116.84 58.42 0) (unit 1)
-    (in_bom yes) (on_board yes)
-    (property "Reference" "J10" (id 0) (at 119.5832 53.8226 0))
-    (property "Value" "Conn_01x02_Male" (id 1) (at 119.5832 56.134 0))
-    (property "Footprint" "Connector_PinHeader_2.54mm:PinHeader_1x02_P2.54mm_Vertical" (id 2) (at 116.84 58.42 0)
-      (effects (font (size 1.27 1.27)) hide)
-    )
-    (property "Datasheet" "~" (id 3) (at 116.84 58.42 0)
-      (effects (font (size 1.27 1.27)) hide)
-    )

Commit message: just before putting vias onto batch18/main
Connections:
- net REG_D: now reaches D6.2 (A), L3.1, Q9.5 (D), Q9.6 (D), Q9.7 (D), Q9.8 (D)
Changed lines of the file:
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@@
   (junction (at 132.08 100.33) (diameter 0) (color 0 0 0 0)
   )
+  (junction (at 71.12 99.06) (diameter 0) (color 0 0 0 0)
+  )
   (junction (at 167.64 100.33) (diameter 0) (color 0 0 0 0)
   )
@@
   )
   (wire (pts (xy 208.28 80.01) (xy 210.82 80.01))
+    (stroke (width 0) (type default) (color 0 0 0 0))
+  )
+  (wire (pts (xy 71.12 99.06) (xy 73.66 99.06))
     (stroke (width 0) (type default) (color 0 0 0 0))
   )
@@
     (effects (font (size 1.27 1.27)) (justify right))
   )
+  (hierarchical_label "REG_D" (shape input) (at 73.66 99.06 0)
+    (effects (font (size 1.27 1.27)) (justify left))
+  )
   (hierarchical_label "PEL_BLK" (shape input) (at 147.32 106.68 180)
