File: kicad/Ninja/batch18/main/file3V3.kicad_sch (KiCad schematic)
At the start: 13 parts, among them U16 CJT1117-3.3, U17 MCP1755T-3302E_OT, U22 MCP1755T-3302E_DC

Commit message: apply changes from Lite
Parts:
- removed C34: 100pF, Capacitor_SMD:C_0603_1608Metric, symbol Device:C
- removed U16: CJT1117-3.3, Package_TO_SOT_SMD:SOT-223, symbol Ninja-qPCR:CJT1117-3.3
- removed U22: MCP1755T-3302E_DC, Package_TO_SOT_SMD:SOT-223-6, symbol Ninja-qPCR:MCP1755T-3302E_DC
- added U7: REG_TO252-3, Ninja-qPCR:REG_TO252-3, symbol Ninja-qPCR:REG_TO252-3
Connections:
- net 12V: now also U7.1 (VIN); no longer C27.1, C29.1, C31.1, U17.1 (VIN), U17.3 (SHDN)
- net 3V3D: now also U7.2 (VOUT)
- net GND: now also U7.3 (GND)
- net PWRGD: no longer names the net of U17.4 (PWRGD)
- new net 5V_UPS: C27.1, C29.1, C31.1, U17.1 (VIN), U17.3 (SHDN)
- no-connect marks 0 -> 1
Other:
- note added: "150mA LDO"
- note removed: "500mA LDO"

Commit message: batch18/main schematic done
Parts:
- added U9: LD1086DTTR, Package_TO_SOT_SMD:SOT-223, symbol Regulator_Linear:LD1086DTTR
Connections:
- net 12V: now also U9.3 (IN)
- net 3V3D: now also U9.2 (OUT)
- net GND: now also U9.1 (ADJ/GND)
Changed lines of the file:
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@@
+    (stroke (width 0) (type default) (color 0 0 0 0))
+  )
+  (wire (pts (xy 134.874 139.7) (xy 137.16 139.7))
     (stroke (width 0) (type default) (color 0 0 0 0))
   )
@@
     (stroke (width 0) (type default) (color 0 0 0 0))
   )
+  (wire (pts (xy 147.32 147.32) (xy 147.32 149.352))
+    (stroke (width 0) (type default) (color 0 0 0 0))
+  )
   (wire (pts (xy 200.66 71.12) (xy 200.66 77.47))
     (stroke (width 0) (type default) (color 0 0 0 0))
@@
   )
   (wire (pts (xy 156.21 105.41) (xy 163.83 105.41))
+    (stroke (width 0) (type default) (color 0 0 0 0))
+  )
+  (wire (pts (xy 157.48 139.7) (xy 159.512 139.7))
     (stroke (width 0) (type default) (color 0 0 0 0))
   )
@@
     (effects (font (size 1.27 1.27)) (justify right))
     (property "Intersheet References" "${INTERSHEET_REFS}" (id 0) (at 0 0 0)
+      (effects (font (size 1.27 1.27)) hide)
+    )
+  )
+  (global_label "3V3D" (shape input) (at 159.512 139.7 0) (fields_autoplaced)
+    (effects (font (size 1.27 1.27)) (justify left))
+    (property "Intersheet References" "${INTERSHEET_REFS}" (id 0) (at -24.638 34.29 0)
       (effects (font (size 1.27 1.27)) hide)
     )
@@
     )
   )
+  (global_label "12V" (shape input) (at 134.874 139.7 180) (fields_autoplaced)
+    (effects (font (size 1.27 1.27)) (justify right))
+    (property "Intersheet References" "${INTERSHEET_REFS}" (id 0) (at 37.084 34.29 0)
+      (effects (font (size 1.27 1.27)) hide)
+    )
+  )
   (symbol (lib_id "Device:C") (at 116.84 81.28 0) (unit 1)
     (in_bom yes) (on_board yes)
@@
     )
     (property "Datasheet" "" (id 3) (at 146.05 102.87 0)
+      (effects (font (size 1.27 1.27)) hide)
+    )
+    (pin "1")
+    (pin "2")
+    (pin "3")
+  )
+  (symbol (lib_id "Regulator_Linear:LD1086DTTR") (at 147.32 139.7 0) (unit 1)
+    (in_bom yes) (on_board yes) (fields_autoplaced)
+    (property "Reference" "U9" (id 0) (at 147.32 130.9202 0))
+    (property "Value" "LD1086DTTR" (id 1) (at 147.32 133.4571 0))
+    (property "Footprint" "Package_TO_SOT_SMD:SOT-223" (id 2) (at 147.32 127 0)
+      (effects (font (size 1.27 1.27)) hide)
+    )
+    (property "Datasheet" "https://www.st.com/resource/en/datasheet/ld1086.pdf" (id 3) (at 147.32 127 0)
       (effects (font (size 1.27 1.27)) hide)
     )
@@
     (pin "5")
   )
+  (symbol (lib_id "power:GND") (at 147.32 149.352 0) (unit 1)
+    (in_bom yes) (on_board yes)
+    (property "Reference" "#PWR0118" (id 0) (at 147.32 155.702 0)
+      (effects (font (size 1.27 1.27)) hide)
+    )
+    (property "Value" "GND" (id 1) (at 147.447 153.7462 0))
+    (property "Footprint" "" (id 2) (at 147.32 149.352 0)
+      (effects (font (size 1.27 1.27)) hide)
+    )
+    (property "Datasheet" "" (id 3) (at 147.32 149.352 0)
+      (effects (font (size 1.27 1.27)) hide)
+    )
+    (pin "1")
+  )
 )
