File: kicad/Ninja/batch18/main/qPCR-main.kicad_sch (KiCad schematic)
At the start: 41 parts, among them J1 Barrel_Jack_Switch, J11 Conn_01x01_Male, J19 Conn_01x08_Male, J2 Raspberry_Pi_3A_Plus_wpi, J3 Conn_01x01_Male, J4 Conn_01x01_Male, J5 Conn_01x01_Male, J6 Conn_01x01_Male, J7 Conn_01x01_Male, J8 Conn_01x01_Male, J9 Conn_01x01_Male, Q1 Q_NMOS_GSD, Q10 Q_NPN_BCE, Q2 Q_NMOS_GSD, Q3 Q_NMOS_GSD, Q4 Q_NPN_BCE, Q5 Q_NMOS_GSD, Q6 Q_NPN_BCE, SW1 SW_Reed, U5 DIN4_PWR

Commit message: renamed
Other:
- note added: "NOTE: MUX_SELECT/MUX_SELECT_INV replaced @ PhotoMUX"
Changed lines of the file:
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@@
+    (effects (font (size 1.27 1.27)) (justify left bottom))
+  )
+  (text "NOTE: MUX_SELECT/MUX_SELECT_INV replaced @ PhotoMUX"
+    (at 19.05 17.78 0)
     (effects (font (size 1.27 1.27)) (justify left bottom))
   )

Commit message: wiring batch18/main
Parts:
- removed J4, J5, J6: Conn_01x01_Male, Connector_PinHeader_2.54mm:PinHeader_1x01_P2.54mm_Vertical, symbol Connector:Conn_01x01_Male
- J11, J3, J7, J8, J9: footprint Connector_PinHeader_2.54mm:PinHeader_1x01_P2.54mm_Vertical -> Connector_PinHeader_1.27mm:PinHeader_1x01_P1.27mm_Vertical
Connections:
- net GPIO14: no longer J2.23 (GPIO14/SCLK)
- net MUX_SELECT: now also J2.23 (GPIO14/SCLK); no longer J2.22 (GPIO6)
- net GPIO12 renamed LED_SPI_MOSI
- net GPIO13 renamed LED_BLANK
- net GPIO5 renamed LED_SPI_SCLK
- new net LED_LAT: J2.22 (GPIO6)
Other:
- removed sheet -1V
- moved on the sheet: J11, J3

Commit message: apply changes from Lite
Parts:
- removed D7: LED_GBAR, LED_THT:LED_D5.0mm-4_RGB, symbol Device:LED_GBAR
- removed J7: Conn_01x01_Male, Connector_PinHeader_1.27mm:PinHeader_1x01_P1.27mm_Vertical, symbol Connector:Conn_01x01_Male
- removed Q10, Q4, Q6: Q_NPN_BCE, Package_TO_SOT_SMD:SOT-23, symbol Device:Q_NPN_BEC
- removed R20, R38, R39: ?, Resistor_SMD:R_0603_1608Metric, symbol Device:R
- removed R40, R41, R42: 10k, Resistor_SMD:R_0603_1608Metric, symbol Device:R
- added J?: Conn_01x10_Male, symbol Connector:Conn_01x10_Male
Connections:
- net 3V3D: now also J?.1 (Pin_1)
- net 5V_UPS: now also J?.9 (Pin_9)
- net FAN: now also J2.40 (GPIO29); no longer J2.29 (GPIO21)
- net GND: now also J?.4 (Pin_4), J?.5 (Pin_5)
- net GPIO22: no longer J2.31 (GPIO22)
- net GPIO29: no longer J2.40 (GPIO29)
- net GPIO3: no longer J2.15 (GPIO3)
- net GPIO7: no longer J2.7 (GPIO7)
- net I2C_SCL: now also J?.2 (Pin_2)
- net I2C_SDA: now also J?.3 (Pin_3)
- net THERM_R_SWITCH: now also J2.15 (GPIO3); no longer J2.26 (GPIO11/CE1)
- net ADC_DRDY renamed LED
- net LED: now also J?.10 (Pin_10)
- new net NAU_DRDY: J2.7 (GPIO7)
- new net TACT1: J2.26 (GPIO11/CE1), J?.8 (Pin_8)
- new net TACT2: J2.29 (GPIO21), J?.7 (Pin_7)
- new net TACT3: J2.31 (GPIO22), J?.6 (Pin_6)
Other:
- note removed: "NOTE: MUX_SELECT/MUX_SELECT_INV replaced @ PhotoMUX"

Commit message: batch18/main schematic done
Parts:
- J5: renamed from J?; footprint (none) -> Connector_PinHeader_2.54mm:PinHeader_1x10_P2.54mm_Vertical
Connections:
- net 5V_UPS: now also J5.8 (Pin_8); no longer J5.9 (Pin_9)
- net GND: now also J5.10 (Pin_10); no longer J5.5 (Pin_5)
- net LED: now also J5.9 (Pin_9); no longer J5.10 (Pin_10)
- net TACT1: now also J5.7 (Pin_7); no longer J5.8 (Pin_8)
- net TACT2: now also J5.6 (Pin_6); no longer J5.7 (Pin_7)
- net TACT3: now also J5.5 (Pin_5); no longer J5.6 (Pin_6)

Commit message: batch18/main schematic done
Parts:
- removed J11, J3, J8, J9: Conn_01x01_Male, Connector_PinHeader_1.27mm:PinHeader_1x01_P1.27mm_Vertical, symbol Connector:Conn_01x01_Male
Other:
- sheet 5V_UPS renamed Power
- removed sheet 3V3

Commit message: wired batch03/main
Connections:
- net 3V3D: now also J5.4 (Pin_4); no longer J5.1 (Pin_1)
- net 5V_UPS: now also J5.1 (Pin_1); no longer J5.8 (Pin_8)
- net GND: now also J5.2 (Pin_2), J5.3 (Pin_3); no longer J5.10 (Pin_10), J5.4 (Pin_4)
- net I2C_SCL: now also J5.5 (Pin_5); no longer J5.2 (Pin_2)
- net I2C_SDA: now also J5.6 (Pin_6); no longer J5.3 (Pin_3)
- net LED: now also J5.10 (Pin_10); no longer J5.9 (Pin_9)
- net TACT1: now also J5.9 (Pin_9); no longer J5.7 (Pin_7)
- net TACT2: now also J5.8 (Pin_8); no longer J5.6 (Pin_6)
- net TACT3: now also J5.7 (Pin_7); no longer J5.5 (Pin_5)
