File: kicad/Ninja/batch18/main/filePhotoThermistors.kicad_sch (KiCad schematic)
At the start: 10 parts, among them U6 SN74LV4051A, U8 TS12A12511DCNR

Commit message: batch18/main schematic done
Parts:
- TLID1, TWELL1: footprint Connector_PinHeader_2.54mm:PinHeader_1x02_P2.54mm_Vertical -> Connector_Hirose:Hirose_DF13-02P-1.25DSA_1x02_P1.25mm_Vertical
Changed lines of the file:
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@@
     (property "Reference" "TLID1" (id 0) (at 257.81 64.77 0))
     (property "Value" "Conn_01x02_Male" (id 1) (at 264.16 67.31 0))
-    (property "Footprint" "Connector_PinHeader_2.54mm:PinHeader_1x02_P2.54mm_Vertical" (id 2) (at 254 64.77 0)
+    (property "Footprint" "Connector_Hirose:Hirose_DF13-02P-1.25DSA_1x02_P1.25mm_Vertical" (id 2) (at 254 64.77 0)
       (effects (font (size 1.27 1.27)) hide)
     )
@@
     (property "Reference" "TWELL1" (id 0) (at 257.81 49.53 0))
     (property "Value" "Conn_01x02_Male" (id 1) (at 264.16 52.07 0))
-    (property "Footprint" "Connector_PinHeader_2.54mm:PinHeader_1x02_P2.54mm_Vertical" (id 2) (at 254 49.53 0)
+    (property "Footprint" "Connector_Hirose:Hirose_DF13-02P-1.25DSA_1x02_P1.25mm_Vertical" (id 2) (at 254 49.53 0)
       (effects (font (size 1.27 1.27)) hide)
     )

Commit message: just before wiring photo-(single|dual)
Parts:
- U8: footprint Package_TO_SOT_SMD:SOT-23-8 -> Ninja-qPCR:SOT-23-8-8.3mil
Changed lines of the file:
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@@
       (effects (font (size 1.524 1.524)))
     )
-    (property "Footprint" "Package_TO_SOT_SMD:SOT-23-8" (id 2) (at 64.77 85.344 0)
+    (property "Footprint" "Ninja-qPCR:SOT-23-8-8.3mil" (id 2) (at 64.77 85.344 0)
       (effects (font (size 1.524 1.524)) hide)
     )
