File: kicad/Ninja/batch19/photo-dual/photo-dual.kicad_sch (KiCad schematic)
At the start: 21 parts, among them J1 Conn_01x60_Male

Commit message: wired batch19/photo-dual
Parts:
- removed TH1: Thermistor, Resistors_SMD:R_0603_HandSoldering, symbol Device:Thermistor
- added D10B1, D11B1, D12B1, D13B1, D14B1, D15B1, D16B1, D1B1, D2B1, D3B1, D4B1, D5B1, D6B1, D7B1, D8B1, D9B1: D_Photo, Ninja-qPCR:D_1206_nosilk, symbol Device:D_Photo
- D10A1, D11A1, D12A1, D13A1, D14A1, D15A1, D16A1, D1A1, D2A1, D3A1, D4A1, D5A1, D6A1, D7A1, D8A1, D9A1: footprint Ninja-qPCR:SFH2200_2201_2240 -> Ninja-qPCR:D_1206_nosilk
Connections:
- net N_PD_OUT1: no longer J1.51 (Pin_51)
- net N_PD_OUT11: no longer J1.56 (Pin_56)
- net N_PD_OUT13: no longer J1.57 (Pin_57)
- net N_PD_OUT15: no longer J1.58 (Pin_58)
- net N_PD_OUT3: no longer J1.52 (Pin_52)
- net N_PD_OUT5: no longer J1.53 (Pin_53)
- net N_PD_OUT7: no longer J1.54 (Pin_54)
- net N_PD_OUT9: no longer J1.55 (Pin_55)
- net S_PD_OUT1: no longer J1.50 (Pin_50)
- net S_PD_OUT11: no longer J1.45 (Pin_45)
- net S_PD_OUT13: no longer J1.44 (Pin_44)
- net S_PD_OUT15: no longer J1.43 (Pin_43)
- net S_PD_OUT3: no longer J1.49 (Pin_49)
- net S_PD_OUT5: no longer J1.48 (Pin_48)
- net S_PD_OUT7: no longer J1.47 (Pin_47)
- net S_PD_OUT9: no longer J1.46 (Pin_46)
- net VCCA: now also D10B1.1 (K), D11B1.1 (K), D12B1.1 (K), D13B1.1 (K), D14B1.1 (K), D15B1.1 (K), D16B1.1 (K), D1B1.1 (K), D2B1.1 (K), D3B1.1 (K), D4B1.1 (K), D5B1.1 (K), D6B1.1 (K), D7B1.1 (K), D8B1.1 (K), D9B1.1 (K)
- net TH2: now reaches J1.41 (Pin_41), TH2.1
- net TH2: now also J1.42 (Pin_42)
- new net N_PD_OUT10: D5B1.2 (A), J1.55 (Pin_55)
- new net N_PD_OUT12: D6B1.2 (A), J1.56 (Pin_56)
- new net N_PD_OUT14: D7B1.2 (A), J1.57 (Pin_57)
- new net N_PD_OUT16: D8B1.2 (A), J1.58 (Pin_58)
- new net N_PD_OUT2: D1B1.2 (A), J1.51 (Pin_51)
- new net N_PD_OUT4: D2B1.2 (A), J1.52 (Pin_52)
- new net N_PD_OUT6: D3B1.2 (A), J1.53 (Pin_53)
- new net N_PD_OUT8: D4B1.2 (A), J1.54 (Pin_54)
- new net S_PD_OUT10: D13B1.2 (A), J1.46 (Pin_46)
- new net S_PD_OUT12: D14B1.2 (A), J1.45 (Pin_45)
- new net S_PD_OUT14: D15B1.2 (A), J1.44 (Pin_44)
- new net S_PD_OUT16: D16B1.2 (A), J1.43 (Pin_43)
- new net S_PD_OUT2: D9B1.2 (A), J1.50 (Pin_50)
- new net S_PD_OUT4: D10B1.2 (A), J1.49 (Pin_49)
- new net S_PD_OUT6: D11B1.2 (A), J1.48 (Pin_48)
- new net S_PD_OUT8: D12B1.2 (A), J1.47 (Pin_47)
