File: kicad/Ninja/batch19/led-north/qPCR-led-north.kicad_pcb (KiCad board)
At the start: 2 copper layers, 123.1 x 17.3 mm, 11 parts, among them U1 Conn_01x10_Male, U2 Conn_01x10_Male

Commit message: batch19 changes
Parts:
- removed U2: Conn_01x10_Male, Pin_Headers:Pin_Header_Angled_2x05_Pitch2.54mm
- U1: footprint Connector_PinSocket_2.54mm:PinSocket_1x10_P2.54mm_Horizontal -> Connector_PinHeader_1.27mm:PinHeader_2x05_P1.27mm_Horizontal
- moved U1 5.30 mm to (186.1, 101.4), turned to -90 degrees
- moved C1 3.89 mm to (185.1, 99.4), turned to 180 degrees
Routing:
- net GND: track 348.8 -> 3.77 mm, vias 113 -> 119
- net OUT14: track 150.2 -> 39.9 mm
- net OUT9: track 0.00 -> 86.7 mm, vias 0 -> 1
- net OUT13: track 96.1 -> 45.7 mm, vias 2 -> 0
- net OUT10: track 59.1 -> 83.4 mm
- net OUT12: track 83.9 -> 63.6 mm, vias 0 -> 1
- net VCC: track 120.9 -> 101.2 mm, vias 2 -> 0
- net OUT15: track 33.6 -> 26.2 mm, vias 2 -> 0
- net OUT11: track 72.2 -> 66.4 mm, vias 2 -> 0
- net OUT16: track 20.1 -> 18.0 mm, vias 1 -> 0
Other:
- board size 123.1 x 17.3 mm -> 98.5 x 16.6 mm
- board text added: "98.5x16.6mm"
- board text added: "batch19/led-north"
- board text removed: "121.5x16.6mm"
- board text removed: "batch16/led-north"
